File: LabPowerSupply/LabPowerSupply.kicad_sch (KiCad schematic)
At the start: 2 parts

Commit message: more work
Other:
- added sheet No Connect (NoConnect.kicad_sch)

Commit message: Resistor footprints changed to 0603
Parts:
- Mains1: value Conn_01x02 -> (none); footprint Connector_TE-Connectivity:TE_MATE-N-LOK_1-770866-x_1x02_P4.14mm_Vertical -> (none)
- Transformer1: value FS24-800-C2 -> (none); footprint SamacSys_Parts:FS24800C2 -> (none)

Commit message: Added mcu capacitors, split 5v inductors
Parts:
- Mains1: value (none) -> Conn_01x02; footprint (none) -> Connector_TE-Connectivity:TE_MATE-N-LOK_1-770866-x_1x02_P4.14mm_Vertical
- Transformer1: value (none) -> FS24-800-C2; footprint (none) -> SamacSys_Parts:FS24800C2
Changed lines of the file:
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@@
     (in_bom yes) (on_board yes) (fields_autoplaced)
     (property "Reference" "Mains1" (id 0) (at 46.99 88.9 0))
-    (property "Value" "" (id 1) (at 46.99 91.44 0))
-    (property "Footprint" "" (id 2) (at 46.99 95.25 0)
+    (property "Value" "Conn_01x02" (id 1) (at 46.99 91.44 0))
+    (property "Footprint" "Connector_TE-Connectivity:TE_MATE-N-LOK_1-770866-x_1x02_P4.14mm_Vertical" (id 2) (at 46.99 95.25 0)
       (effects (font (size 1.27 1.27)) hide)
     )
@@
     (in_bom yes) (on_board yes) (fields_autoplaced)
     (property "Reference" "Transformer1" (id 0) (at 71.12 86.36 0))
-    (property "Value" "" (id 1) (at 71.12 88.9 0))
-    (property "Footprint" "" (id 2) (at 83.82 91.44 0)
+    (property "Value" "FS24-800-C2" (id 1) (at 71.12 88.9 0))
+    (property "Footprint" "SamacSys_Parts:FS24800C2" (id 2) (at 83.82 91.44 0)
       (effects (font (size 1.27 1.27)) (justify left) hide)
     )
@@
     )
     (path "/08fd45d5-b4ab-46e8-a348-5c4ac8e52155/bcce49d6-fd1a-44d3-995e-3240f3f7d1d9"
-      (reference "C1_Power1") (unit 1) (value "100n") (footprint "Capacitor_THT:C_Disc_D5.0mm_W2.5mm_P2.50mm")
+      (reference "C1_Power1") (unit 1) (value "1u") (footprint "Capacitor_THT:C_Disc_D5.0mm_W2.5mm_P2.50mm")
     )
     (path "/67b0d6de-a54b-4bd2-af78-b383bfe8d0e6/2fe31ecc-dee4-4c05-8775-22bca1687116"
-      (reference "C1_Power2") (unit 1) (value "100n") (footprint "Capacitor_THT:C_Disc_D5.0mm_W2.5mm_P2.50mm")
+      (reference "C1_Power2") (unit 1) (value "1u") (footprint "Capacitor_THT:C_Disc_D5.0mm_W2.5mm_P2.50mm")
     )
     (path "/0c3af00c-caea-46d1-9953-712c4efb6180/4d9e571f-dae1-4ed5-9f8d-0fc03fa434f7/a5f06dfc-3fa8-40e8-bc3f-73cb2d658cb7"
@@
     )
     (path "/08fd45d5-b4ab-46e8-a348-5c4ac8e52155/bcb7596c-c3bf-4311-8160-e481c5cfbf72"
-      (reference "C2_Power1") (unit 1) (value "100n") (footprint "Capacitor_THT:C_Disc_D5.0mm_W2.5mm_P2.50mm")
+      (reference "C2_Power1") (unit 1) (value "1u") (footprint "Capacitor_THT:C_Disc_D5.0mm_W2.5mm_P2.50mm")
     )
     (path "/67b0d6de-a54b-4bd2-af78-b383bfe8d0e6/89c3d81a-415d-4e4f-8aca-b9a43e4ea4e6"
-      (reference "C2_Power2") (unit 1) (value "100n") (footprint "Capacitor_THT:C_Disc_D5.0mm_W2.5mm_P2.50mm")
+      (reference "C2_Power2") (unit 1) (value "1u") (footprint "Capacitor_THT:C_Disc_D5.0mm_W2.5mm_P2.50mm")
     )
     (path "/0c3af00c-caea-46d1-9953-712c4efb6180/4d9e571f-dae1-4ed5-9f8d-0fc03fa434f7/c2401621-782c-4840-972a-334269bd565e"
@@
     )
     (path "/08fd45d5-b4ab-46e8-a348-5c4ac8e52155/fba723df-b241-4063-8db6-e899e6f4ff70"
-      (reference "C3_Power1") (unit 1) (value "100n") (footprint "Capacitor_THT:C_Disc_D5.0mm_W2.5mm_P2.50mm")
+      (reference "C3_Power1") (unit 1) (value "1u") (footprint "Capacitor_THT:C_Disc_D5.0mm_W2.5mm_P2.50mm")
     )
     (path "/67b0d6de-a54b-4bd2-af78-b383bfe8d0e6/a057987a-fac2-41b8-b2c2-daf0bc999920"
-      (reference "C3_Power2") (unit 1) (value "100n") (footprint "Capacitor_THT:C_Disc_D5.0mm_W2.5mm_P2.50mm")
+      (reference "C3_Power2") (unit 1) (value "1u") (footprint "Capacitor_THT:C_Disc_D5.0mm_W2.5mm_P2.50mm")
     )
     (path "/0c3af00c-caea-46d1-9953-712c4efb6180/4d9e571f-dae1-4ed5-9f8d-0fc03fa434f7/2ed3a93c-6d90-4a89-a9b9-d1e7f7ad9b38"
@@
     )
     (path "/08fd45d5-b4ab-46e8-a348-5c4ac8e52155/5c06a03a-cb7e-42fc-97a3-9252db7bc734"
-      (reference "C4_Power1") (unit 1) (value "100n") (footprint "Capacitor_THT:C_Disc_D5.0mm_W2.5mm_P2.50mm")
+      (reference "C4_Power1") (unit 1) (value "1u") (footprint "Capacitor_THT:C_Disc_D5.0mm_W2.5mm_P2.50mm")
     )
     (path "/67b0d6de-a54b-4bd2-af78-b383bfe8d0e6/c11229af-7317-4a21-9101-b04d4349c67e"
-      (reference "C4_Power2") (unit 1) (value "100n") (footprint "Capacitor_THT:C_Disc_D5.0mm_W2.5mm_P2.50mm")
+      (reference "C4_Power2") (unit 1) (value "1u") (footprint "Capacitor_THT:C_Disc_D5.0mm_W2.5mm_P2.50mm")
     )
     (path "/0c3af00c-caea-46d1-9953-712c4efb6180/4d9e571f-dae1-4ed5-9f8d-0fc03fa434f7/e38e77b8-dfbe-4d6f-8f9a-1469db9af726"
@@
     )
     (path "/08fd45d5-b4ab-46e8-a348-5c4ac8e52155/73ed34cb-2319-423d-a2d9-b56cfdb9a478"
-      (reference "C5_Power1") (unit 1) (value "100n") (footprint "Capacitor_THT:C_Disc_D5.0mm_W2.5mm_P2.50mm")
+      (reference "C5_Power1") (unit 1) (value "1u") (footprint "Capacitor_THT:C_Disc_D5.0mm_W2.5mm_P2.50mm")
+    )
+    (path "/67b0d6de-a54b-4bd2-af78-b383bfe8d0e6/40b71e71-4082-40ca-a69a-009671993fc3"
+      (reference "C5_Power2") (unit 1) (value "100n") (footprint "Capacitor_THT:C_Disc_D5.0mm_W2.5mm_P2.50mm")
+    )
+    (path "/08fd45d5-b4ab-46e8-a348-5c4ac8e52155/bd5a79c6-aa46-4103-8d4f-d3095a27715e"
+      (reference "C6_Power1") (unit 1) (value "100n") (footprint "Capacitor_THT:C_Disc_D5.0mm_W2.5mm_P2.50mm")
+    )
+    (path "/67b0d6de-a54b-4bd2-af78-b383bfe8d0e6/564c12e1-207b-44cf-ac13-5c637ab497bd"
+      (reference "C6_Power2") (unit 1) (value "100n") (footprint "Capacitor_THT:C_Disc_D5.0mm_W2.5mm_P2.50mm")
+    )
+    (path "/08fd45d5-b4ab-46e8-a348-5c4ac8e52155/cd1edf3b-3e7c-43bc-a516-57c87c49d787"
+      (reference "C7_Power1") (unit 1) (value "100n") (footprint "Capacitor_THT:C_Disc_D5.0mm_W2.5mm_P2.50mm")
+    )
+    (path "/67b0d6de-a54b-4bd2-af78-b383bfe8d0e6/19841d47-ab65-4d53-b3c2-70f6cd47d3cc"
+      (reference "C7_Power2") (unit 1) (value "100n") (footprint "Capacitor_THT:C_Disc_D5.0mm_W2.5mm_P2.50mm")
+    )
+    (path "/08fd45d5-b4ab-46e8-a348-5c4ac8e52155/5ce2b538-e262-444d-8a0d-ae353703919a"
+      (reference "C8_Power1") (unit 1) (value "100n") (footprint "Capacitor_THT:C_Disc_D5.0mm_W2.5mm_P2.50mm")
+    )
+    (path "/67b0d6de-a54b-4bd2-af78-b383bfe8d0e6/0407b42a-0ddf-4f4e-af6d-6a2d762e7e74"
+      (reference "C8_Power2") (unit 1) (value "100n") (footprint "Capacitor_THT:C_Disc_D5.0mm_W2.5mm_P2.50mm")
+    )
+    (path "/08fd45d5-b4ab-46e8-a348-5c4ac8e52155/a8ac00b1-09cf-406c-89ac-9cb9c31c44f4"
+      (reference "C9_Power1") (unit 1) (value "100n") (footprint "Capacitor_THT:C_Disc_D5.0mm_W2.5mm_P2.50mm")
+    )
+    (path "/08fd45d5-b4ab-46e8-a348-5c4ac8e52155/da229d01-fa09-4a32-8b11-399c27e22ee5"
+      (reference "C10_Power1") (unit 1) (value "100n") (footprint "Capacitor_THT:C_Disc_D5.0mm_W2.5mm_P2.50mm")
     )
     (path "/77fcffa2-9d70-4da1-b633-0d00734b5fc1/204e8e4f-f461-4b9c-b352-ebb2dcedd771"
@@
       (reference "OpAmp1") (unit 3) (value "LM324") (footprint "Package_DIP:DIP-14_W7.62mm")
     )
+    (path "/0c3af00c-caea-46d1-9953-712c4efb6180/7e152100-3451-4635-9914-2a0b75d7b7b6/c98ac8c9-2ce6-4f4f-a66b-643b63dca01e"
+      (reference "OpAmp1") (unit 4) (value "LM324") (footprint "Package_DIP:DIP-14_W7.62mm")
+    )
     (path "/0c3af00c-caea-46d1-9953-712c4efb6180/7e152100-3451-4635-9914-2a0b75d7b7b6/501b9250-99c9-4da3-9fc2-a388092a2dd4"
       (reference "OpAmp1") (unit 5) (value "LM324") (footprint "Package_DIP:DIP-14_W7.62mm")
@@
       (reference "OpAmp2") (unit 3) (value "LM324") (footprint "Package_DIP:DIP-14_W7.62mm")
     )
+    (path "/e157f35d-29d6-4a10-895b-6361f5380fc1/7e152100-3451-4635-9914-2a0b75d7b7b6/c98ac8c9-2ce6-4f4f-a66b-643b63dca01e"
+      (reference "OpAmp2") (unit 4) (value "LM324") (footprint "Package_DIP:DIP-14_W7.62mm")
+    )
     (path "/e157f35d-29d6-4a10-895b-6361f5380fc1/7e152100-3451-4635-9914-2a0b75d7b7b6/501b9250-99c9-4da3-9fc2-a388092a2dd4"
       (reference "OpAmp2") (unit 5) (value "LM324") (footprint "Package_DIP:DIP-14_W7.62mm")
@@
       (reference "Q_CP2") (unit 1) (value "2N2219") (footprint "Package_TO_SOT_THT:TO-92_Inline")
     )
+    (path "/08fd45d5-b4ab-46e8-a348-5c4ac8e52155/d0a03699-50f8-46bd-ab34-900d57d3ac72"
+      (reference "R1_Boot1") (unit 1) (value "5.1k") (footprint "Resistor_SMD:R_0603_1608Metric")
+    )
+    (path "/67b0d6de-a54b-4bd2-af78-b383bfe8d0e6/20fdca4d-bd4e-4bc0-bd45-9561394615ec"
+      (reference "R1_Boot2") (unit 1) (value "5.1k") (footprint "Resistor_SMD:R_0603_1608Metric")
+    )
     (path "/0c3af00c-caea-46d1-9953-712c4efb6180/877b38b4-9fca-4c7e-a1c5-d7e6e745bcaf/47bd2c18-6728-4952-aff4-c44e64d63302"
       (reference "R1_CS1") (unit 1) (value "300m") (footprint "Resistor_SMD:R_0603_1608Metric")
@@
       (reference "R1_SVR2") (unit 1) (value "180m") (footprint "Resistor_SMD:R_0603_1608Metric")
     )
+    (path "/08fd45d5-b4ab-46e8-a348-5c4ac8e52155/cf13ead1-ddae-4fa6-9727-c15c5a0ceb3a"
+      (reference "R2_Boot1") (unit 1) (value "5.1k") (footprint "Resistor_SMD:R_0603_1608Metric")
+    )
+    (path "/67b0d6de-a54b-4bd2-af78-b383bfe8d0e6/0cdb8c3e-f721-4add-89d6-3f0786c7cbca"
+      (reference "R2_Boot2") (unit 1) (value "5.1k") (footprint "Resistor_SMD:R_0603_1608Metric")
+    )
     (path "/0c3af00c-caea-46d1-9953-712c4efb6180/877b38b4-9fca-4c7e-a1c5-d7e6e745bcaf/8df2c858-0b30-453b-9770-4c5e8393702b"
       (reference "R2_CS1") (unit 1) (value "3k") (footprint "Resistor_SMD:R_0603_1608Metric")
@@
       (reference "R10_OA2") (unit 1) (value "1k") (footprint "Resistor_SMD:R_0603_1608Metric")
     )
-    (path "/08fd45d5-b4ab-46e8-a348-5c4ac8e52155/d0a03699-50f8-46bd-ab34-900d57d3ac72"
-      (reference "R_Boot1") (unit 1) (value "5.1k") (footprint "Resistor_SMD:R_0603_1608Metric")
-    )
-    (path "/67b0d6de-a54b-4bd2-af78-b383bfe8d0e6/20fdca4d-bd4e-4bc0-bd45-9561394615ec"
-      (reference "R_Boot2") (unit 1) (value "5.1k") (footprint "Resistor_SMD:R_0603_1608Metric")
+    (path "/0c3af00c-caea-46d1-9953-712c4efb6180/7e152100-3451-4635-9914-2a0b75d7b7b6/9e40d895-a947-4b33-a248-0d0dda788e56"
+      (reference "R11_OA1") (unit 1) (value "4k") (footprint "Resistor_SMD:R_0603_1608Metric")
+    )
+    (path "/e157f35d-29d6-4a10-895b-6361f5380fc1/7e152100-3451-4635-9914-2a0b75d7b7b6/9e40d895-a947-4b33-a248-0d0dda788e56"
+      (reference "R11_OA2") (unit 1) (value "4k") (footprint "Resistor_SMD:R_0603_1608Metric")
     )
     (path "/08fd45d5-b4ab-46e8-a348-5c4ac8e52155/b78ed596-2ebf-471d-87f7-c16705ddf1d3"
