File: LabPowerSupply/ChargePump.kicad_sch (KiCad schematic)
At the start: 9 parts

Commit message: in the middle
Parts:
- Q_CP1: value 2N2219 -> FMNT495TA; footprint Package_TO_SOT_THT:TO-92_Inline -> Package_TO_SOT_SMD:SOT-23
Changed lines of the file:
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@@
       (effects (font (size 1.27 1.27)) (justify left))
     )
-    (property "Value" "2N2219" (id 1) (at 189.23 107.9499 0)
+    (property "Value" "FMNT495TA" (id 1) (at 189.23 107.9499 0)
       (effects (font (size 1.27 1.27)) (justify left))
     )
-    (property "Footprint" "Package_TO_SOT_THT:TO-92_Inline" (id 2) (at 189.23 104.775 0)
+    (property "Footprint" "Package_TO_SOT_SMD:SOT-23" (id 2) (at 189.23 104.775 0)
       (effects (font (size 1.27 1.27) italic) (justify left) hide)
     )
