File: LabPowerSupply/ChargePump.kicad_sch (KiCad schematic)
At the start: 9 parts

Commit message: Start tallying
Parts:
- Q_CP1: footprint (none) -> Package_TO_SOT_SMD:SOT-23
Changed lines of the file:
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@@
       (effects (font (size 1.27 1.27)) (justify left))
     )
-    (property "Footprint" "" (id 2) (at 189.23 104.775 0)
+    (property "Footprint" "Package_TO_SOT_SMD:SOT-23" (id 2) (at 189.23 104.775 0)
       (effects (font (size 1.27 1.27) italic) (justify left) hide)
     )

Commit message: almost done
Parts:
- removed Q_CP1: 2N2219, Package_TO_SOT_SMD:SOT-23, symbol Transistor_BJT:2N2219
Other:
- moved on the sheet: R_CP1
Changed lines of the file:
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@@
     (stroke (width 0) (type default) (color 0 0 0 0))
   )
-  (wire (pts (xy 184.15 100.33) (xy 191.77 100.33))
+  (wire (pts (xy 187.96 100.33) (xy 191.77 100.33))
     (stroke (width 0) (type default) (color 0 0 0 0))
   )
@@
   )
   (wire (pts (xy 128.27 109.22) (xy 128.27 111.76))
+    (stroke (width 0) (type default) (color 0 0 0 0))
+  )
+  (wire (pts (xy 180.34 100.33) (xy 176.53 100.33))
     (stroke (width 0) (type default) (color 0 0 0 0))
   )
@@
     (pin "2")
   )
-  (symbol (lib_id "Transistor_BJT:2N2219") (at 194.31 106.68 180) (unit 1)
-    (in_bom yes) (on_board yes) (fields_autoplaced)
-    (property "Reference" "Q_CP1" (id 0) (at 189.23 105.4099 0)
-      (effects (font (size 1.27 1.27)) (justify left))
-    )
-    (property "Value" "2N2219" (id 1) (at 189.23 107.9499 0)
-      (effects (font (size 1.27 1.27)) (justify left))
-    )
-    (property "Footprint" "Package_TO_SOT_SMD:SOT-23" (id 2) (at 189.23 104.775 0)
-      (effects (font (size 1.27 1.27) italic) (justify left) hide)
-    )
-    (property "Datasheet" "http://www.onsemi.com/pub_link/Collateral/2N2219-D.PDF" (id 3) (at 194.31 106.68 0)
-      (effects (font (size 1.27 1.27)) (justify left) hide)
-    )
-    (pin "1")
-    (pin "2")
-    (pin "3")
-  )
   (symbol (lib_id "Diode:1N4001") (at 137.16 100.33 0) (unit 1)
     (in_bom yes) (on_board yes)
@@
     (pin "2")
   )
-  (symbol (lib_id "Device:R_US") (at 180.34 100.33 90) (unit 1)
+  (symbol (lib_id "Device:R_US") (at 184.15 100.33 90) (unit 1)
     (in_bom yes) (on_board yes) (fields_autoplaced)
-    (property "Reference" "R_CP1" (id 0) (at 180.34 93.98 90))
-    (property "Value" "1k" (id 1) (at 180.34 96.52 90))
-    (property "Footprint" "Resistor_SMD:R_0603_1608Metric" (id 2) (at 180.594 99.314 90)
+    (property "Reference" "R_CP1" (id 0) (at 184.15 93.98 90))
+    (property "Value" "1k" (id 1) (at 184.15 96.52 90))
+    (property "Footprint" "Resistor_SMD:R_0603_1608Metric" (id 2) (at 184.404 99.314 90)
       (effects (font (size 1.27 1.27)) hide)
     )
-    (property "Datasheet" "~" (id 3) (at 180.34 100.33 0)
+    (property "Datasheet" "~" (id 3) (at 184.15 100.33 0)
       (effects (font (size 1.27 1.27)) hide)
     )

Commit message: Changed capacitors to x7r
Parts:
- C1_CP1, C2_CP1, C3_CP1, C4_CP1: footprint Capacitor_SMD:C_0805_2012Metric -> Capacitor_SMD:C_1210_3225Metric
Changed lines of the file:
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@@
       (effects (font (size 1.27 1.27)) (justify left))
     )
-    (property "Footprint" "Capacitor_SMD:C_0805_2012Metric" (id 2) (at 145.7452 111.76 0)
+    (property "Footprint" "Capacitor_SMD:C_1210_3225Metric" (id 2) (at 145.7452 111.76 0)
       (effects (font (size 1.27 1.27)) hide)
     )
@@
     (property "Reference" "C1_CP1" (id 0) (at 123.19 92.71 90))
     (property "Value" "22u" (id 1) (at 123.19 95.25 90))
-    (property "Footprint" "Capacitor_SMD:C_0805_2012Metric" (id 2) (at 127 99.3648 0)
+    (property "Footprint" "Capacitor_SMD:C_1210_3225Metric" (id 2) (at 127 99.3648 0)
       (effects (font (size 1.27 1.27)) hide)
     )
@@
       (effects (font (size 1.27 1.27)) (justify left))
     )
-    (property "Footprint" "Capacitor_SMD:C_0805_2012Metric" (id 2) (at 159.7152 111.76 0)
+    (property "Footprint" "Capacitor_SMD:C_1210_3225Metric" (id 2) (at 159.7152 111.76 0)
       (effects (font (size 1.27 1.27)) hide)
     )
@@
     (property "Reference" "C2_CP1" (id 0) (at 123.19 81.28 90))
     (property "Value" "22u" (id 1) (at 123.19 83.82 90))
-    (property "Footprint" "Capacitor_SMD:C_0805_2012Metric" (id 2) (at 127 87.9348 0)
+    (property "Footprint" "Capacitor_SMD:C_1210_3225Metric" (id 2) (at 127 87.9348 0)
       (effects (font (size 1.27 1.27)) hide)
     )

Commit message: SMD Oscillator
Parts:
- added Q1_CP1: FMMT495TA, Package_TO_SOT_SMD:SOT-23, symbol Transistor_BJT:PN2222A
Connections:
- net Charge: now also Q1_CP1.3 (C)
- net GND: now also Q1_CP1.2 (B)
- net at R_CP1.2: now also Q1_CP1.1 (E)
Changed lines of the file:
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@@
     (pin "2")
   )
+  (symbol (lib_id "Transistor_BJT:PN2222A") (at 194.31 106.68 180) (unit 1)
+    (in_bom yes) (on_board yes) (fields_autoplaced)
+    (property "Reference" "Q1_CP1" (id 0) (at 189.23 105.4099 0)
+      (effects (font (size 1.27 1.27)) (justify left))
+    )
+    (property "Value" "FMMT495TA" (id 1) (at 189.23 107.9499 0)
+      (effects (font (size 1.27 1.27)) (justify left))
+    )
+    (property "Footprint" "Package_TO_SOT_SMD:SOT-23" (id 2) (at 189.23 104.775 0)
+      (effects (font (size 1.27 1.27) italic) (justify left) hide)
+    )
+    (property "Datasheet" "https://www.onsemi.com/pub/Collateral/PN2222-D.PDF" (id 3) (at 194.31 106.68 0)
+      (effects (font (size 1.27 1.27)) (justify left) hide)
+    )
+    (pin "1")
+    (pin "2")
+    (pin "3")
+  )
 )

Commit message: Updated Part List
Parts:
- C1_CP1, C2_CP1, C3_CP1, C4_CP1: value 22u -> (none); footprint Capacitor_SMD:C_1210_3225Metric -> (none)
- C5_CP1: value 1m -> (none); footprint Capacitor_THT:CP_Radial_D10.0mm_P5.00mm -> (none)
- D1_CP1, D2_CP1: value 1N4001 -> (none); footprint Diode_SMD:D_SMA -> (none)
- Q1_CP1: value FMMT495TA -> (none); footprint Package_TO_SOT_SMD:SOT-23 -> (none)
- R_CP1: value 1k -> (none); footprint Resistor_SMD:R_0603_1608Metric -> (none)
Changed lines of the file:
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@@
       (effects (font (size 1.27 1.27)) (justify left))
     )
-    (property "Value" "22u" (id 1) (at 148.59 109.2199 0)
+    (property "Value" "" (id 1) (at 148.59 109.2199 0)
       (effects (font (size 1.27 1.27)) (justify left))
     )
-    (property "Footprint" "Capacitor_SMD:C_1210_3225Metric" (id 2) (at 145.7452 111.76 0)
+    (property "Footprint" "" (id 2) (at 145.7452 111.76 0)
       (effects (font (size 1.27 1.27)) hide)
     )
@@
     (in_bom yes) (on_board yes) (fields_autoplaced)
     (property "Reference" "C1_CP1" (id 0) (at 123.19 92.71 90))
-    (property "Value" "22u" (id 1) (at 123.19 95.25 90))
-    (property "Footprint" "Capacitor_SMD:C_1210_3225Metric" (id 2) (at 127 99.3648 0)
+    (property "Value" "" (id 1) (at 123.19 95.25 90))
+    (property "Footprint" "" (id 2) (at 127 99.3648 0)
       (effects (font (size 1.27 1.27)) hide)
     )
@@
       (effects (font (size 1.27 1.27)) (justify left))
     )
-    (property "Value" "22u" (id 1) (at 162.56 109.2199 0)
+    (property "Value" "" (id 1) (at 162.56 109.2199 0)
       (effects (font (size 1.27 1.27)) (justify left))
     )
-    (property "Footprint" "Capacitor_SMD:C_1210_3225Metric" (id 2) (at 159.7152 111.76 0)
+    (property "Footprint" "" (id 2) (at 159.7152 111.76 0)
       (effects (font (size 1.27 1.27)) hide)
     )
@@
       (effects (font (size 1.27 1.27)) (justify right))
     )
-    (property "Value" "1N4001" (id 1) (at 134.62 106.68 90))
-    (property "Footprint" "Diode_SMD:D_SMA" (id 2) (at 132.715 105.41 0)
+    (property "Value" "" (id 1) (at 134.62 106.68 90))
+    (property "Footprint" "" (id 2) (at 132.715 105.41 0)
       (effects (font (size 1.27 1.27)) hide)
     )
@@
     (in_bom yes) (on_board yes) (fields_autoplaced)
     (property "Reference" "C2_CP1" (id 0) (at 123.19 81.28 90))
-    (property "Value" "22u" (id 1) (at 123.19 83.82 90))
-    (property "Footprint" "Capacitor_SMD:C_1210_3225Metric" (id 2) (at 127 87.9348 0)
+    (property "Value" "" (id 1) (at 123.19 83.82 90))
+    (property "Footprint" "" (id 2) (at 127 87.9348 0)
       (effects (font (size 1.27 1.27)) hide)
     )
@@
     (in_bom yes) (on_board yes)
     (property "Reference" "D1_CP1" (id 0) (at 136.8425 93.98 0))
-    (property "Value" "1N4001" (id 1) (at 137.16 96.52 0))
-    (property "Footprint" "Diode_SMD:D_SMA" (id 2) (at 137.16 104.775 0)
+    (property "Value" "" (id 1) (at 137.16 96.52 0))
+    (property "Footprint" "" (id 2) (at 137.16 104.775 0)
       (effects (font (size 1.27 1.27)) hide)
     )
@@
       (effects (font (size 1.27 1.27)) (justify right))
     )
-    (property "Value" "1m" (id 1) (at 180.34 113.6649 0)
+    (property "Value" "" (id 1) (at 180.34 113.6649 0)
       (effects (font (size 1.27 1.27)) (justify right))
     )
-    (property "Footprint" "Capacitor_THT:CP_Radial_D10.0mm_P5.00mm" (id 2) (at 176.53 111.76 0)
+    (property "Footprint" "" (id 2) (at 176.53 111.76 0)
       (effects (font (size 1.27 1.27)) hide)
     )
@@
     (in_bom yes) (on_board yes) (fields_autoplaced)
     (property "Reference" "R_CP1" (id 0) (at 184.15 93.98 90))
-    (property "Value" "1k" (id 1) (at 184.15 96.52 90))
-    (property "Footprint" "Resistor_SMD:R_0603_1608Metric" (id 2) (at 184.404 99.314 90)
+    (property "Value" "" (id 1) (at 184.15 96.52 90))
+    (property "Footprint" "" (id 2) (at 184.404 99.314 90)
       (effects (font (size 1.27 1.27)) hide)
     )
@@
       (effects (font (size 1.27 1.27)) (justify left))
     )
-    (property "Value" "FMMT495TA" (id 1) (at 189.23 107.9499 0)
+    (property "Value" "" (id 1) (at 189.23 107.9499 0)
       (effects (font (size 1.27 1.27)) (justify left))
     )
-    (property "Footprint" "Package_TO_SOT_SMD:SOT-23" (id 2) (at 189.23 104.775 0)
+    (property "Footprint" "" (id 2) (at 189.23 104.775 0)
       (effects (font (size 1.27 1.27) italic) (justify left) hide)
     )
