File: LabPowerSupply/PrimaryController.kicad_sch (KiCad schematic)
At the start: 25 parts, among them Y1 8M

Commit message: another commit
Parts:
- C10_Power1, C1_Power1, C2_Power1, C3_Power1, C4_Power1, C5_Power1, C6_Power1, C7_Power1, C8_Power1, C9_Power1: footprint Capacitor_THT:C_Disc_D5.0mm_W2.5mm_P2.50mm -> Capacitor_SMD:C_0603_1608Metric
Changed lines of the file:
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@@
     (property "Reference" "C4_Power1" (id 0) (at 132.08 15.24 90))
     (property "Value" "1u" (id 1) (at 132.08 17.78 90))
-    (property "Footprint" "Capacitor_THT:C_Disc_D5.0mm_W2.5mm_P2.50mm" (id 2) (at 135.89 21.8948 0)
+    (property "Footprint" "Capacitor_SMD:C_0603_1608Metric" (id 2) (at 135.89 21.8948 0)
       (effects (font (size 1.27 1.27)) hide)
     )
@@
     (property "Reference" "C8_Power1" (id 0) (at 120.65 31.75 90))
     (property "Value" "100n" (id 1) (at 120.65 34.29 90))
-    (property "Footprint" "Capacitor_THT:C_Disc_D5.0mm_W2.5mm_P2.50mm" (id 2) (at 124.46 26.9748 0)
+    (property "Footprint" "Capacitor_SMD:C_0603_1608Metric" (id 2) (at 124.46 26.9748 0)
       (effects (font (size 1.27 1.27)) hide)
     )
@@
     (property "Reference" "C5_Power1" (id 0) (at 143.51 15.24 90))
     (property "Value" "1u" (id 1) (at 143.51 17.78 90))
-    (property "Footprint" "Capacitor_THT:C_Disc_D5.0mm_W2.5mm_P2.50mm" (id 2) (at 147.32 21.8948 0)
+    (property "Footprint" "Capacitor_SMD:C_0603_1608Metric" (id 2) (at 147.32 21.8948 0)
       (effects (font (size 1.27 1.27)) hide)
     )
@@
     (property "Reference" "C9_Power1" (id 0) (at 132.08 31.75 90))
     (property "Value" "100n" (id 1) (at 132.08 34.29 90))
-    (property "Footprint" "Capacitor_THT:C_Disc_D5.0mm_W2.5mm_P2.50mm" (id 2) (at 135.89 26.9748 0)
+    (property "Footprint" "Capacitor_SMD:C_0603_1608Metric" (id 2) (at 135.89 26.9748 0)
       (effects (font (size 1.27 1.27)) hide)
     )
@@
     (property "Reference" "C2_Power1" (id 0) (at 109.22 15.24 90))
     (property "Value" "1u" (id 1) (at 109.22 17.78 90))
-    (property "Footprint" "Capacitor_THT:C_Disc_D5.0mm_W2.5mm_P2.50mm" (id 2) (at 113.03 21.8948 0)
+    (property "Footprint" "Capacitor_SMD:C_0603_1608Metric" (id 2) (at 113.03 21.8948 0)
       (effects (font (size 1.27 1.27)) hide)
     )
@@
     (property "Reference" "C1_Power1" (id 0) (at 97.79 15.24 90))
     (property "Value" "1u" (id 1) (at 97.79 17.78 90))
-    (property "Footprint" "Capacitor_THT:C_Disc_D5.0mm_W2.5mm_P2.50mm" (id 2) (at 101.6 21.8948 0)
+    (property "Footprint" "Capacitor_SMD:C_0603_1608Metric" (id 2) (at 101.6 21.8948 0)
       (effects (font (size 1.27 1.27)) hide)
     )
@@
     (property "Reference" "C6_Power1" (id 0) (at 97.79 31.75 90))
     (property "Value" "100n" (id 1) (at 97.79 34.29 90))
-    (property "Footprint" "Capacitor_THT:C_Disc_D5.0mm_W2.5mm_P2.50mm" (id 2) (at 101.6 26.9748 0)
+    (property "Footprint" "Capacitor_SMD:C_0603_1608Metric" (id 2) (at 101.6 26.9748 0)
       (effects (font (size 1.27 1.27)) hide)
     )
@@
     (property "Reference" "C7_Power1" (id 0) (at 109.22 31.75 90))
     (property "Value" "100n" (id 1) (at 109.22 34.29 90))
-    (property "Footprint" "Capacitor_THT:C_Disc_D5.0mm_W2.5mm_P2.50mm" (id 2) (at 113.03 26.9748 0)
+    (property "Footprint" "Capacitor_SMD:C_0603_1608Metric" (id 2) (at 113.03 26.9748 0)
       (effects (font (size 1.27 1.27)) hide)
     )
@@
     (property "Reference" "C10_Power1" (id 0) (at 143.51 31.75 90))
     (property "Value" "100n" (id 1) (at 143.51 34.29 90))
-    (property "Footprint" "Capacitor_THT:C_Disc_D5.0mm_W2.5mm_P2.50mm" (id 2) (at 147.32 26.9748 0)
+    (property "Footprint" "Capacitor_SMD:C_0603_1608Metric" (id 2) (at 147.32 26.9748 0)
       (effects (font (size 1.27 1.27)) hide)
     )
@@
     (property "Reference" "C3_Power1" (id 0) (at 120.65 15.24 90))
     (property "Value" "1u" (id 1) (at 120.65 17.78 90))
-    (property "Footprint" "Capacitor_THT:C_Disc_D5.0mm_W2.5mm_P2.50mm" (id 2) (at 124.46 21.8948 0)
-      (effects (font (size 1.27 1.27)) hide)
-    )
+    (property "Footprint" "Capacitor_SMD:C_0603_1608Metric" (id 2) (at 124.46 21.8948 0)
+      (effects (font (size 1.27 1.27)) hide)
+    )

Commit message: Made oscillator caps smd
Parts:
- C1_Y1, C2_Y1: footprint Capacitor_THT:C_Disc_D5.0mm_W2.5mm_P2.50mm -> (none)
Changed lines of the file:
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@@
     (property "Reference" "C2_Y1" (id 0) (at 90.17 87.63 90))
     (property "Value" "100n" (id 1) (at 90.17 90.17 90))
-    (property "Footprint" "Capacitor_THT:C_Disc_D5.0mm_W2.5mm_P2.50mm" (id 2) (at 93.98 83.5152 0)
+    (property "Footprint" "" (id 2) (at 93.98 83.5152 0)
       (effects (font (size 1.27 1.27)) hide)
     )
@@
     (property "Reference" "C1_Y1" (id 0) (at 82.55 73.66 90))
     (property "Value" "100n" (id 1) (at 82.55 76.2 90))
-    (property "Footprint" "Capacitor_THT:C_Disc_D5.0mm_W2.5mm_P2.50mm" (id 2) (at 93.98 73.9648 0)
+    (property "Footprint" "" (id 2) (at 93.98 73.9648 0)
       (effects (font (size 1.27 1.27)) hide)
     )

Commit message: fixed linear cap footprints
Parts:
- C1_Y1, C2_Y1: footprint (none) -> Capacitor_SMD:C_0603_1608Metric
Changed lines of the file:
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@@
     (property "Reference" "C2_Y1" (id 0) (at 90.17 87.63 90))
     (property "Value" "100n" (id 1) (at 90.17 90.17 90))
-    (property "Footprint" "" (id 2) (at 93.98 83.5152 0)
+    (property "Footprint" "Capacitor_SMD:C_0603_1608Metric" (id 2) (at 93.98 83.5152 0)
       (effects (font (size 1.27 1.27)) hide)
     )
@@
     (property "Reference" "C1_Y1" (id 0) (at 82.55 73.66 90))
     (property "Value" "100n" (id 1) (at 82.55 76.2 90))
-    (property "Footprint" "" (id 2) (at 93.98 73.9648 0)
+    (property "Footprint" "Capacitor_SMD:C_0603_1608Metric" (id 2) (at 93.98 73.9648 0)
       (effects (font (size 1.27 1.27)) hide)
     )

Commit message: Changed most parts to smd
Parts:
- C10_Power1, C1_Power1, C1_Y1, C2_Power1, C2_Y1, C3_Power1, C4_Power1, C5_Power1, C6_Power1, C7_Power1, C8_Power1, C9_Power1: footprint Capacitor_SMD:C_0603_1608Metric -> Capacitor_SMD:C_0805_2012Metric
Changed lines of the file:
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@@
     (property "Reference" "C2_Y1" (id 0) (at 90.17 87.63 90))
     (property "Value" "100n" (id 1) (at 90.17 90.17 90))
-    (property "Footprint" "Capacitor_SMD:C_0603_1608Metric" (id 2) (at 93.98 83.5152 0)
+    (property "Footprint" "Capacitor_SMD:C_0805_2012Metric" (id 2) (at 93.98 83.5152 0)
       (effects (font (size 1.27 1.27)) hide)
     )
@@
     (property "Reference" "C4_Power1" (id 0) (at 132.08 15.24 90))
     (property "Value" "1u" (id 1) (at 132.08 17.78 90))
-    (property "Footprint" "Capacitor_SMD:C_0603_1608Metric" (id 2) (at 135.89 21.8948 0)
+    (property "Footprint" "Capacitor_SMD:C_0805_2012Metric" (id 2) (at 135.89 21.8948 0)
       (effects (font (size 1.27 1.27)) hide)
     )
@@
     (property "Reference" "C8_Power1" (id 0) (at 120.65 31.75 90))
     (property "Value" "100n" (id 1) (at 120.65 34.29 90))
-    (property "Footprint" "Capacitor_SMD:C_0603_1608Metric" (id 2) (at 124.46 26.9748 0)
+    (property "Footprint" "Capacitor_SMD:C_0805_2012Metric" (id 2) (at 124.46 26.9748 0)
       (effects (font (size 1.27 1.27)) hide)
     )
@@
     (property "Reference" "C5_Power1" (id 0) (at 143.51 15.24 90))
     (property "Value" "1u" (id 1) (at 143.51 17.78 90))
-    (property "Footprint" "Capacitor_SMD:C_0603_1608Metric" (id 2) (at 147.32 21.8948 0)
+    (property "Footprint" "Capacitor_SMD:C_0805_2012Metric" (id 2) (at 147.32 21.8948 0)
       (effects (font (size 1.27 1.27)) hide)
     )
@@
     (property "Reference" "C1_Y1" (id 0) (at 82.55 73.66 90))
     (property "Value" "100n" (id 1) (at 82.55 76.2 90))
-    (property "Footprint" "Capacitor_SMD:C_0603_1608Metric" (id 2) (at 93.98 73.9648 0)
+    (property "Footprint" "Capacitor_SMD:C_0805_2012Metric" (id 2) (at 93.98 73.9648 0)
       (effects (font (size 1.27 1.27)) hide)
     )
@@
     (property "Reference" "C9_Power1" (id 0) (at 132.08 31.75 90))
     (property "Value" "100n" (id 1) (at 132.08 34.29 90))
-    (property "Footprint" "Capacitor_SMD:C_0603_1608Metric" (id 2) (at 135.89 26.9748 0)
+    (property "Footprint" "Capacitor_SMD:C_0805_2012Metric" (id 2) (at 135.89 26.9748 0)
       (effects (font (size 1.27 1.27)) hide)
     )
@@
     (property "Reference" "C2_Power1" (id 0) (at 109.22 15.24 90))
     (property "Value" "1u" (id 1) (at 109.22 17.78 90))
-    (property "Footprint" "Capacitor_SMD:C_0603_1608Metric" (id 2) (at 113.03 21.8948 0)
+    (property "Footprint" "Capacitor_SMD:C_0805_2012Metric" (id 2) (at 113.03 21.8948 0)
       (effects (font (size 1.27 1.27)) hide)
     )
@@
     (property "Reference" "C1_Power1" (id 0) (at 97.79 15.24 90))
     (property "Value" "1u" (id 1) (at 97.79 17.78 90))
-    (property "Footprint" "Capacitor_SMD:C_0603_1608Metric" (id 2) (at 101.6 21.8948 0)
+    (property "Footprint" "Capacitor_SMD:C_0805_2012Metric" (id 2) (at 101.6 21.8948 0)
       (effects (font (size 1.27 1.27)) hide)
     )
@@
     (property "Reference" "C6_Power1" (id 0) (at 97.79 31.75 90))
     (property "Value" "100n" (id 1) (at 97.79 34.29 90))
-    (property "Footprint" "Capacitor_SMD:C_0603_1608Metric" (id 2) (at 101.6 26.9748 0)
+    (property "Footprint" "Capacitor_SMD:C_0805_2012Metric" (id 2) (at 101.6 26.9748 0)
       (effects (font (size 1.27 1.27)) hide)
     )
@@
     (property "Reference" "C7_Power1" (id 0) (at 109.22 31.75 90))
     (property "Value" "100n" (id 1) (at 109.22 34.29 90))
-    (property "Footprint" "Capacitor_SMD:C_0603_1608Metric" (id 2) (at 113.03 26.9748 0)
+    (property "Footprint" "Capacitor_SMD:C_0805_2012Metric" (id 2) (at 113.03 26.9748 0)
       (effects (font (size 1.27 1.27)) hide)
     )
@@
     (property "Reference" "C10_Power1" (id 0) (at 143.51 31.75 90))
     (property "Value" "100n" (id 1) (at 143.51 34.29 90))
-    (property "Footprint" "Capacitor_SMD:C_0603_1608Metric" (id 2) (at 147.32 26.9748 0)
+    (property "Footprint" "Capacitor_SMD:C_0805_2012Metric" (id 2) (at 147.32 26.9748 0)
       (effects (font (size 1.27 1.27)) hide)
     )
@@
     (property "Reference" "C3_Power1" (id 0) (at 120.65 15.24 90))
     (property "Value" "1u" (id 1) (at 120.65 17.78 90))
-    (property "Footprint" "Capacitor_SMD:C_0603_1608Metric" (id 2) (at 124.46 21.8948 0)
-      (effects (font (size 1.27 1.27)) hide)
-    )
+    (property "Footprint" "Capacitor_SMD:C_0805_2012Metric" (id 2) (at 124.46 21.8948 0)
+      (effects (font (size 1.27 1.27)) hide)
+    )

Commit message: Fixed oscillator caps, began changing resistors to more common values
Parts:
- C1_Y1, C2_Y1: value 100n -> 20p; footprint Capacitor_SMD:C_0805_2012Metric -> Capacitor_SMD:C_0603_1608Metric
Changed lines of the file:
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@@
   (symbol (lib_id "Device:C") (at 90.17 82.55 90) (mirror x) (unit 1)
     (in_bom yes) (on_board yes)
-    (property "Reference" "C2_Y1" (id 0) (at 90.17 87.63 90))
-    (property "Value" "100n" (id 1) (at 90.17 90.17 90))
-    (property "Footprint" "Capacitor_SMD:C_0805_2012Metric" (id 2) (at 93.98 83.5152 0)
+    (property "Reference" "C2_Y1" (id 0) (at 82.55 81.28 90))
+    (property "Value" "20p" (id 1) (at 82.55 83.82 90))
+    (property "Footprint" "Capacitor_SMD:C_0603_1608Metric" (id 2) (at 93.98 83.5152 0)
       (effects (font (size 1.27 1.27)) hide)
     )
@@
     (in_bom yes) (on_board yes)
     (property "Reference" "C1_Y1" (id 0) (at 82.55 73.66 90))
-    (property "Value" "100n" (id 1) (at 82.55 76.2 90))
-    (property "Footprint" "Capacitor_SMD:C_0805_2012Metric" (id 2) (at 93.98 73.9648 0)
+    (property "Value" "20p" (id 1) (at 82.55 76.2 90))
+    (property "Footprint" "Capacitor_SMD:C_0603_1608Metric" (id 2) (at 93.98 73.9648 0)
       (effects (font (size 1.27 1.27)) hide)
     )

Commit message: in the middle
Parts:
- removed J_I2C1: Conn_01x03_Male, Connector_PinHeader_2.54mm:PinHeader_1x03_P2.54mm_Vertical, symbol Connector:Conn_01x03_Male
- added J_I2C: Conn_01x03_Male, Connector_JST:JST_PH_B4B-PH-K_1x04_P2.00mm_Vertical, symbol Connector:Conn_01x04_Male
Connections:
- net GND: now also J_I2C.1 (Pin_1)
- net I2C SCL: now also J_I2C.4 (Pin_4)
- net I2C SDA: now also J_I2C.3 (Pin_3)
- new net 5 Volts: J_I2C.2 (Pin_2)
Changed lines of the file:
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@@
   (junction (at 93.98 82.55) (diameter 0) (color 0 0 0 0)
   )
-  (junction (at 180.34 130.81) (diameter 0) (color 0 0 0 0)
-  )
   (junction (at 105.41 22.86) (diameter 0) (color 0 0 0 0)
   )
@@
   )
   (junction (at 125.73 130.81) (diameter 0) (color 0 0 0 0)
+  )
+  (junction (at 170.18 130.81) (diameter 0) (color 0 0 0 0)
   )
   (junction (at 33.02 158.75) (diameter 0) (color 0 0 0 0)
@@
     (stroke (width 0) (type default) (color 0 0 0 0))
   )
-  (wire (pts (xy 125.73 130.81) (xy 180.34 130.81))
-    (stroke (width 0) (type default) (color 0 0 0 0))
-  )
   (wire (pts (xy 135.89 59.69) (xy 138.43 59.69))
     (stroke (width 0) (type default) (color 0 0 0 0))
@@
     (stroke (width 0) (type default) (color 0 0 0 0))
   )
-  (wire (pts (xy 180.34 107.95) (xy 180.34 130.81))
-    (stroke (width 0) (type default) (color 0 0 0 0))
-  )
   (wire (pts (xy 80.01 161.29) (xy 93.98 161.29))
     (stroke (width 0) (type default) (color 0 0 0 0))
@@
     (stroke (width 0) (type default) (color 0 0 0 0))
   )
+  (wire (pts (xy 170.18 130.81) (xy 205.74 130.81))
+    (stroke (width 0) (type default) (color 0 0 0 0))
+  )
   (wire (pts (xy 33.02 158.75) (xy 67.31 158.75))
     (stroke (width 0) (type default) (color 0 0 0 0))
@@
     (stroke (width 0) (type default) (color 0 0 0 0))
   )
-  (wire (pts (xy 180.34 130.81) (xy 205.74 130.81))
+  (wire (pts (xy 125.73 130.81) (xy 170.18 130.81))
     (stroke (width 0) (type default) (color 0 0 0 0))
   )
@@
     (stroke (width 0) (type default) (color 0 0 0 0))
   )
+  (wire (pts (xy 170.18 97.79) (xy 170.18 130.81))
+    (stroke (width 0) (type default) (color 0 0 0 0))
+  )
   (wire (pts (xy 149.86 36.83) (xy 149.86 25.4))
     (stroke (width 0) (type default) (color 0 0 0 0))
@@
   )
   (wire (pts (xy 205.74 82.55) (xy 205.74 130.81))
+    (stroke (width 0) (type default) (color 0 0 0 0))
+  )
+  (wire (pts (xy 180.34 97.79) (xy 170.18 97.79))
     (stroke (width 0) (type default) (color 0 0 0 0))
   )
@@
   (hierarchical_label "DAC 1" (shape output) (at 138.43 57.15 0)
     (effects (font (size 1.27 1.27)) (justify left))
+  )
+  (hierarchical_label "5 Volts" (shape input) (at 180.34 100.33 180)
+    (effects (font (size 1.27 1.27)) (justify right))
+  )
+  (symbol (lib_id "Connector:Conn_01x04_Male") (at 185.42 100.33 0) (mirror y) (unit 1)
+    (in_bom yes) (on_board yes) (fields_autoplaced)
+    (property "Reference" "J_I2C" (id 0) (at 186.69 100.3299 0)
+      (effects (font (size 1.27 1.27)) (justify right))
+    )
+    (property "Value" "Conn_01x03_Male" (id 1) (at 186.69 102.8699 0)
+      (effects (font (size 1.27 1.27)) (justify right))
+    )
+    (property "Footprint" "Connector_JST:JST_PH_B4B-PH-K_1x04_P2.00mm_Vertical" (id 2) (at 185.42 100.33 0)
+      (effects (font (size 1.27 1.27)) hide)
+    )
+    (property "Datasheet" "~" (id 3) (at 185.42 100.33 0)
+      (effects (font (size 1.27 1.27)) hide)
+    )
+    (pin "1")
+    (pin "2")
+    (pin "3")
+    (pin "4")
   )
   (symbol (lib_id "Device:Crystal") (at 93.98 78.74 90) (unit 1)
@@
       (effects (font (size 1.27 1.27)) hide)
     )
-    (pin "1")
-    (pin "2")
-    (pin "3")
-  )
-  (symbol (lib_id "Connector:Conn_01x03_Male") (at 185.42 105.41 0) (mirror y) (unit 1)
-    (in_bom yes) (on_board yes) (fields_autoplaced)
-    (property "Reference" "J_I2C1" (id 0) (at 186.69 104.1399 0)
-      (effects (font (size 1.27 1.27)) (justify right))
-    )
-    (property "Value" "Conn_01x03_Male" (id 1) (at 186.69 106.6799 0)
-      (effects (font (size 1.27 1.27)) (justify right))
-    )
-    (property "Footprint" "Connector_PinHeader_2.54mm:PinHeader_1x03_P2.54mm_Vertical" (id 2) (at 185.42 105.41 0)
-      (effects (font (size 1.27 1.27)) hide)
-    )
-    (property "Datasheet" "~" (id 3) (at 185.42 105.41 0)
-      (effects (font (size 1.27 1.27)) hide)
-    )

Commit message: Merge
Parts:
- removed J_I2C: Conn_01x03_Male, Connector_JST:JST_PH_B4B-PH-K_1x04_P2.00mm_Vertical, symbol Connector:Conn_01x04_Male
- added J_I2C1: Conn_01x03_Male, Connector_PinHeader_2.54mm:PinHeader_1x03_P2.54mm_Vertical, symbol Connector:Conn_01x03_Male
Connections:
- net GND: now also J_I2C1.3 (Pin_3)
- net I2C SCL: now also J_I2C1.2 (Pin_2)
- net I2C SDA: now also J_I2C1.1 (Pin_1)
Changed lines of the file:
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@@
   (junction (at 93.98 82.55) (diameter 0) (color 0 0 0 0)
   )
+  (junction (at 180.34 130.81) (diameter 0) (color 0 0 0 0)
+  )
   (junction (at 105.41 22.86) (diameter 0) (color 0 0 0 0)
   )
@@
   )
   (junction (at 125.73 130.81) (diameter 0) (color 0 0 0 0)
-  )
-  (junction (at 170.18 130.81) (diameter 0) (color 0 0 0 0)
   )
   (junction (at 33.02 158.75) (diameter 0) (color 0 0 0 0)
@@
     (stroke (width 0) (type default) (color 0 0 0 0))
   )
+  (wire (pts (xy 125.73 130.81) (xy 180.34 130.81))
+    (stroke (width 0) (type default) (color 0 0 0 0))
+  )
   (wire (pts (xy 135.89 59.69) (xy 138.43 59.69))
     (stroke (width 0) (type default) (color 0 0 0 0))
@@
     (stroke (width 0) (type default) (color 0 0 0 0))
   )
+  (wire (pts (xy 180.34 107.95) (xy 180.34 130.81))
+    (stroke (width 0) (type default) (color 0 0 0 0))
+  )
   (wire (pts (xy 80.01 161.29) (xy 93.98 161.29))
     (stroke (width 0) (type default) (color 0 0 0 0))
@@
     (stroke (width 0) (type default) (color 0 0 0 0))
   )
-  (wire (pts (xy 170.18 130.81) (xy 205.74 130.81))
-    (stroke (width 0) (type default) (color 0 0 0 0))
-  )
   (wire (pts (xy 33.02 158.75) (xy 67.31 158.75))
     (stroke (width 0) (type default) (color 0 0 0 0))
@@
     (stroke (width 0) (type default) (color 0 0 0 0))
   )
-  (wire (pts (xy 125.73 130.81) (xy 170.18 130.81))
+  (wire (pts (xy 180.34 130.81) (xy 205.74 130.81))
     (stroke (width 0) (type default) (color 0 0 0 0))
   )
@@
     (stroke (width 0) (type default) (color 0 0 0 0))
   )
-  (wire (pts (xy 170.18 97.79) (xy 170.18 130.81))
-    (stroke (width 0) (type default) (color 0 0 0 0))
-  )
   (wire (pts (xy 149.86 36.83) (xy 149.86 25.4))
     (stroke (width 0) (type default) (color 0 0 0 0))
@@
   )
   (wire (pts (xy 205.74 82.55) (xy 205.74 130.81))
-    (stroke (width 0) (type default) (color 0 0 0 0))
-  )
-  (wire (pts (xy 180.34 97.79) (xy 170.18 97.79))
     (stroke (width 0) (type default) (color 0 0 0 0))
   )
@@
   (hierarchical_label "DAC 1" (shape output) (at 138.43 57.15 0)
     (effects (font (size 1.27 1.27)) (justify left))
-  )
-  (hierarchical_label "5 Volts" (shape input) (at 180.34 100.33 180)
-    (effects (font (size 1.27 1.27)) (justify right))
-  )
-  (symbol (lib_id "Connector:Conn_01x04_Male") (at 185.42 100.33 0) (mirror y) (unit 1)
-    (in_bom yes) (on_board yes) (fields_autoplaced)
-    (property "Reference" "J_I2C" (id 0) (at 186.69 100.3299 0)
-      (effects (font (size 1.27 1.27)) (justify right))
-    )
-    (property "Value" "Conn_01x03_Male" (id 1) (at 186.69 102.8699 0)
-      (effects (font (size 1.27 1.27)) (justify right))
-    )
-    (property "Footprint" "Connector_JST:JST_PH_B4B-PH-K_1x04_P2.00mm_Vertical" (id 2) (at 185.42 100.33 0)
-      (effects (font (size 1.27 1.27)) hide)
-    )
-    (property "Datasheet" "~" (id 3) (at 185.42 100.33 0)
-      (effects (font (size 1.27 1.27)) hide)
-    )
-    (pin "1")
-    (pin "2")
-    (pin "3")
-    (pin "4")
   )
   (symbol (lib_id "Device:Crystal") (at 93.98 78.74 90) (unit 1)
@@
       (effects (font (size 1.27 1.27)) hide)
     )
+    (pin "1")
+    (pin "2")
+    (pin "3")
+  )
+  (symbol (lib_id "Connector:Conn_01x03_Male") (at 185.42 105.41 0) (mirror y) (unit 1)
+    (in_bom yes) (on_board yes) (fields_autoplaced)
+    (property "Reference" "J_I2C1" (id 0) (at 186.69 104.1399 0)
+      (effects (font (size 1.27 1.27)) (justify right))
+    )
+    (property "Value" "Conn_01x03_Male" (id 1) (at 186.69 106.6799 0)
+      (effects (font (size 1.27 1.27)) (justify right))
+    )
+    (property "Footprint" "Connector_PinHeader_2.54mm:PinHeader_1x03_P2.54mm_Vertical" (id 2) (at 185.42 105.41 0)
+      (effects (font (size 1.27 1.27)) hide)
+    )
+    (property "Datasheet" "~" (id 3) (at 185.42 105.41 0)
+      (effects (font (size 1.27 1.27)) hide)
+    )

Commit message: Start tallying
Parts:
- removed Front_Panel1: Conn_02x10_Counter_Clockwise, Connector_IDC:IDC-Header_2x10_P2.54mm_Vertical, symbol Connector_Generic:Conn_02x10_Counter_Clockwise
- removed J_I2C1, J_STLink1: Conn_01x03_Male, Connector_PinHeader_2.54mm:PinHeader_1x03_P2.54mm_Vertical, symbol Connector:Conn_01x03_Male
- added Front_Panel?: Conn_02x10_Counter_Clockwise, Connector_IDC:IDC-Header_2x10_P2.54mm_Vertical, symbol Connector_Generic:Conn_02x08_Counter_Clockwise
- added J_I2C1: Conn_01x03_Male, Connector_PinHeader_2.54mm:PinHeader_1x03_P2.54mm_Vertical, symbol Connector:Conn_01x04_Male
- added J_STLink1: Conn_01x03_Male, Connector_PinHeader_2.54mm:PinHeader_1x03_P2.54mm_Vertical, symbol Connector:Conn_01x05_Male
- renumbered R2_Boot1 to R1_Boot1, R1_Boot1 to R2_Boot1
Connections:
- net 3.3 Volts: now also Front_Panel?.1 (Pin_1), J_STLink1.1 (Pin_1)
- net GND: now also Front_Panel?.5 (Pin_5), J_I2C1.1 (Pin_1), J_STLink1.2 (Pin_2)
- net I2C SCL: now also J_I2C1.4 (Pin_4)
- net I2C SDA: now also J_I2C1.3 (Pin_3)
- net SWCLK: now also J_STLink1.4 (Pin_4)
- net SWDIO: now also J_STLink1.3 (Pin_3)
- net at MCU_1.29 (PB10): now also Front_Panel?.16 (Pin_16)
- net at MCU_1.56 (PB4): now also Front_Panel?.7 (Pin_7)
- net at MCU_1.55 (PB3): now also Front_Panel?.6 (Pin_6)
- net at MCU_1.28 (PB2): now also Front_Panel?.4 (Pin_4)
- net at MCU_1.27 (PB1): now also Front_Panel?.3 (Pin_3)
- net at MCU_1.26 (PB0): now also Front_Panel?.2 (Pin_2)
- net at MCU_1.30 (PB11): now also Front_Panel?.15 (Pin_15)
- net at MCU_1.33 (PB12): now also Front_Panel?.14 (Pin_14)
- net at MCU_1.34 (PB13): now also Front_Panel?.13 (Pin_13)
- net at MCU_1.35 (PB14): now also Front_Panel?.12 (Pin_12)
- net at MCU_1.37 (PC6): now also Front_Panel?.11 (Pin_11)
- net at MCU_1.38 (PC7): now also Front_Panel?.10 (Pin_10)
- net at MCU_1.39 (PC8): now also Front_Panel?.9 (Pin_9)
- net at MCU_1.40 (PC9): now also Front_Panel?.8 (Pin_8)
- net Reset: now reaches MCU_1.7 (NRST), R_Reset1.2, SW_Reset1.3 (B), SW_Reset1.4 (B)
- net Reset: now also J_STLink1.5 (Pin_5)
- new net 5 Volts: J_I2C1.2 (Pin_2)
- no-connect marks 21 -> 24
