File: LabPowerSupply/LabPowerSupply.kicad_pcb (KiCad board)
At the start: 2 copper layers, 216 parts, among them Q1_LVR1 PJA3404_R1_00001, Q1_LVR2 PJA3404_R1_00001, Q2_LVR1 PJA3404_R1_00001, Q2_LVR2 PJA3404_R1_00001, Q3_LVR1 PJA3404_R1_00001, Q3_LVR2 PJA3404_R1_00001, SW11 Decimal, SW12 0, SW13 Backspace, SW14 Current 2, SW15 Cancel, SW21 1, SW22 2, SW23 3, SW24 Voltage 2, SW25 Confirm, SW31 4, SW32 5, SW33 6, SW34 Current 1, SW35 Channel 2, SW41 7, SW42 8, SW43 9, SW44 Voltage 1, SW45 Channel 1, Y1 8M, Y2 8M

Commit message: Made BJT SMD
Parts:
- Q_CP1, Q_CP2: footprint Package_TO_SOT_THT:TO-92_Inline -> Package_TO_SOT_SMD:SOT-23
Changed lines of the file:
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@@
     )
   )
-  (footprint "Package_TO_SOT_THT:TO-92_Inline" (layer "F.Cu")
+  (footprint "Package_TO_SOT_SMD:SOT-23" (layer "F.Cu")
     (at 162.56 63.42 -90)
-    (descr "TO-92 leads in-line, narrow, oval pads, drill 0.75mm (see NXP sot054_po.pdf)")
-    (tags "to-92 sc-43 sc-43a sot54 PA33 transistor")
+    (descr "SOT, 3 Pin (https://www.jedec.org/system/files/docs/to-236h.pdf variant AB), generated with kicad-footprint-generator ipc_gullwing_generator.py")
+    (tags "SOT TO_SOT_SMD")
     (property "Sheetfile" "ChargePump.kicad_sch")
     (property "Sheetname" "Charge Pump")
-    (attr through_hole)
-    (fp_text reference "Q_CP1" (at 1.27 -3.56 90) (layer "F.SilkS")
-      (effects (font (size 1 1) (thickness 0.15)))
-    )
-    (fp_text value "2N2219" (at 1.27 2.79 90) (layer "F.Fab")
-      (effects (font (size 1 1) (thickness 0.15)))
-    )
-    (fp_text user "${REFERENCE}" (at 1.27 0 90) (layer "F.Fab")
-      (effects (font (size 1 1) (thickness 0.15)))
-    )
-    (fp_line (start -0.53 1.85) (end 3.07 1.85) (layer "F.SilkS") (width 0.12))
-    (fp_arc (start -0.568478 1.838478) (mid -1.132087 -0.994977) (end 1.27 -2.6) (layer "F.SilkS") (width 0.12))
-    (fp_arc (start 1.27 -2.6) (mid 3.672087 -0.994977) (end 3.108478 1.838478) (layer "F.SilkS") (width 0.12))
-    (fp_line (start 4 2.01) (end 4 -2.73) (layer "F.CrtYd") (width 0.05))
-    (fp_line (start 4 2.01) (end -1.46 2.01) (layer "F.CrtYd") (width 0.05))
-    (fp_line (start -1.46 -2.73) (end -1.46 2.01) (layer "F.CrtYd") (width 0.05))
-    (fp_line (start -1.46 -2.73) (end 4 -2.73) (layer "F.CrtYd") (width 0.05))
-    (fp_line (start -0.5 1.75) (end 3 1.75) (layer "F.Fab") (width 0.1))
-    (fp_arc (start -0.483625 1.753625) (mid -1.021221 -0.949055) (end 1.27 -2.48) (layer "F.Fab") (width 0.1))
-    (fp_arc (start 1.27 -2.48) (mid 3.561221 -0.949055) (end 3.023625 1.753625) (layer "F.Fab") (width 0.1))
-    (pad "1" thru_hole rect (at 0 0 270) (size 1.05 1.5) (drill 0.75) (layers *.Cu *.Mask)
+    (attr smd)
+    (fp_text reference "Q_CP1" (at 0 -2.4 -90) (layer "F.SilkS")
+      (effects (font (size 1 1) (thickness 0.15)))
+    )
+    (fp_text value "2N2219" (at 0 2.4 -90) (layer "F.Fab")
+      (effects (font (size 1 1) (thickness 0.15)))
+    )
+    (fp_text user "${REFERENCE}" (at 0 0 -90) (layer "F.Fab")
+      (effects (font (size 0.32 0.32) (thickness 0.05)))
+    )
+    (fp_line (start 0 -1.56) (end 0.65 -1.56) (layer "F.SilkS") (width 0.12))
+    (fp_line (start 0 1.56) (end 0.65 1.56) (layer "F.SilkS") (width 0.12))
+    (fp_line (start 0 1.56) (end -0.65 1.56) (layer "F.SilkS") (width 0.12))
+    (fp_line (start 0 -1.56) (end -1.675 -1.56) (layer "F.SilkS") (width 0.12))
+    (fp_line (start -1.92 1.7) (end 1.92 1.7) (layer "F.CrtYd") (width 0.05))
+    (fp_line (start -1.92 -1.7) (end -1.92 1.7) (layer "F.CrtYd") (width 0.05))
+    (fp_line (start 1.92 1.7) (end 1.92 -1.7) (layer "F.CrtYd") (width 0.05))
+    (fp_line (start 1.92 -1.7) (end -1.92 -1.7) (layer "F.CrtYd") (width 0.05))
+    (fp_line (start -0.65 -1.125) (end -0.325 -1.45) (layer "F.Fab") (width 0.1))
+    (fp_line (start -0.325 -1.45) (end 0.65 -1.45) (layer "F.Fab") (width 0.1))
+    (fp_line (start 0.65 -1.45) (end 0.65 1.45) (layer "F.Fab") (width 0.1))
+    (fp_line (start -0.65 1.45) (end -0.65 -1.125) (layer "F.Fab") (width 0.1))
+    (fp_line (start 0.65 1.45) (end -0.65 1.45) (layer "F.Fab") (width 0.1))
+    (pad "1" smd roundrect (at -0.9375 -0.95 270) (size 1.475 0.6) (layers "F.Cu" "F.Paste" "F.Mask") (roundrect_rratio 0.25)
       (net 175 "Net-(Q_CP1-Pad1)") (pinfunction "E") (pintype "passive"))
-    (pad "2" thru_hole oval (at 1.27 0 270) (size 1.05 1.5) (drill 0.75) (layers *.Cu *.Mask)
+    (pad "2" smd roundrect (at -0.9375 0.95 270) (size 1.475 0.6) (layers "F.Cu" "F.Paste" "F.Mask") (roundrect_rratio 0.25)
       (net 13 "GND1") (pinfunction "B") (pintype "passive"))
-    (pad "3" thru_hole oval (at 2.54 0 270) (size 1.05 1.5) (drill 0.75) (layers *.Cu *.Mask)
+    (pad "3" smd roundrect (at 0.9375 0 270) (size 1.475 0.6) (layers "F.Cu" "F.Paste" "F.Mask") (roundrect_rratio 0.25)
       (net 24 "/Channel Power Supply 1/Charge Pump/Charge") (pinfunction "C") (pintype "passive"))
-    (model "${KICAD6_3DMODEL_DIR}/Package_TO_SOT_THT.3dshapes/TO-92_Inline.wrl"
+    (model "${KICAD6_3DMODEL_DIR}/Package_TO_SOT_SMD.3dshapes/SOT-23.wrl"
       (offset (xyz 0 0 0))
       (scale (xyz 1 1 1))
@@
     )
   )
-  (footprint "Package_TO_SOT_THT:TO-92_Inline" (layer "F.Cu")
+  (footprint "Package_TO_SOT_SMD:SOT-23" (layer "F.Cu")
     (at 154.94 104.14 -90)
-    (descr "TO-92 leads in-line, narrow, oval pads, drill 0.75mm (see NXP sot054_po.pdf)")
-    (tags "to-92 sc-43 sc-43a sot54 PA33 transistor")
+    (descr "SOT, 3 Pin (https://www.jedec.org/system/files/docs/to-236h.pdf variant AB), generated with kicad-footprint-generator ipc_gullwing_generator.py")
+    (tags "SOT TO_SOT_SMD")
     (property "Sheetfile" "ChargePump.kicad_sch")
     (property "Sheetname" "Charge Pump")
-    (attr through_hole)
-    (fp_text reference "Q_CP2" (at 1.27 -3.56 90) (layer "F.SilkS")
-      (effects (font (size 1 1) (thickness 0.15)))
-    )
-    (fp_text value "2N2219" (at 1.27 2.79 90) (layer "F.Fab")
-      (effects (font (size 1 1) (thickness 0.15)))
-    )
-    (fp_text user "${REFERENCE}" (at 1.27 0 90) (layer "F.Fab")
-      (effects (font (size 1 1) (thickness 0.15)))
-    )
-    (fp_line (start -0.53 1.85) (end 3.07 1.85) (layer "F.SilkS") (width 0.12))
-    (fp_arc (start -0.568478 1.838478) (mid -1.132087 -0.994977) (end 1.27 -2.6) (layer "F.SilkS") (width 0.12))
-    (fp_arc (start 1.27 -2.6) (mid 3.672087 -0.994977) (end 3.108478 1.838478) (layer "F.SilkS") (width 0.12))
-    (fp_line (start 4 2.01) (end -1.46 2.01) (layer "F.CrtYd") (width 0.05))
-    (fp_line (start -1.46 -2.73) (end -1.46 2.01) (layer "F.CrtYd") (width 0.05))
-    (fp_line (start 4 2.01) (end 4 -2.73) (layer "F.CrtYd") (width 0.05))
-    (fp_line (start -1.46 -2.73) (end 4 -2.73) (layer "F.CrtYd") (width 0.05))
-    (fp_line (start -0.5 1.75) (end 3 1.75) (layer "F.Fab") (width 0.1))
-    (fp_arc (start 1.27 -2.48) (mid 3.561221 -0.949055) (end 3.023625 1.753625) (layer "F.Fab") (width 0.1))
-    (fp_arc (start -0.483625 1.753625) (mid -1.021221 -0.949055) (end 1.27 -2.48) (layer "F.Fab") (width 0.1))
-    (pad "1" thru_hole rect (at 0 0 270) (size 1.05 1.5) (drill 0.75) (layers *.Cu *.Mask)
+    (attr smd)
+    (fp_text reference "Q_CP2" (at 0 -2.4 -90) (layer "F.SilkS")
+      (effects (font (size 1 1) (thickness 0.15)))
+    )
+    (fp_text value "2N2219" (at 0 2.4 -90) (layer "F.Fab")
+      (effects (font (size 1 1) (thickness 0.15)))
+    )
+    (fp_text user "${REFERENCE}" (at 0 0 -90) (layer "F.Fab")
+      (effects (font (size 0.32 0.32) (thickness 0.05)))
+    )
+    (fp_line (start 0 -1.56) (end -1.675 -1.56) (layer "F.SilkS") (width 0.12))
+    (fp_line (start 0 1.56) (end -0.65 1.56) (layer "F.SilkS") (width 0.12))
+    (fp_line (start 0 1.56) (end 0.65 1.56) (layer "F.SilkS") (width 0.12))
+    (fp_line (start 0 -1.56) (end 0.65 -1.56) (layer "F.SilkS") (width 0.12))
+    (fp_line (start -1.92 -1.7) (end -1.92 1.7) (layer "F.CrtYd") (width 0.05))
+    (fp_line (start 1.92 1.7) (end 1.92 -1.7) (layer "F.CrtYd") (width 0.05))
+    (fp_line (start 1.92 -1.7) (end -1.92 -1.7) (layer "F.CrtYd") (width 0.05))
+    (fp_line (start -1.92 1.7) (end 1.92 1.7) (layer "F.CrtYd") (width 0.05))
+    (fp_line (start -0.65 -1.125) (end -0.325 -1.45) (layer "F.Fab") (width 0.1))
+    (fp_line (start 0.65 -1.45) (end 0.65 1.45) (layer "F.Fab") (width 0.1))
+    (fp_line (start -0.325 -1.45) (end 0.65 -1.45) (layer "F.Fab") (width 0.1))
+    (fp_line (start 0.65 1.45) (end -0.65 1.45) (layer "F.Fab") (width 0.1))
+    (fp_line (start -0.65 1.45) (end -0.65 -1.125) (layer "F.Fab") (width 0.1))
+    (pad "1" smd roundrect (at -0.9375 -0.95 270) (size 1.475 0.6) (layers "F.Cu" "F.Paste" "F.Mask") (roundrect_rratio 0.25)
       (net 191 "Net-(Q_CP2-Pad1)") (pinfunction "E") (pintype "passive"))
-    (pad "2" thru_hole oval (at 1.27 0 270) (size 1.05 1.5) (drill 0.75) (layers *.Cu *.Mask)
+    (pad "2" smd roundrect (at -0.9375 0.95 270) (size 1.475 0.6) (layers "F.Cu" "F.Paste" "F.Mask") (roundrect_rratio 0.25)
       (net 8 "GND2") (pinfunction "B") (pintype "passive"))
-    (pad "3" thru_hole oval (at 2.54 0 270) (size 1.05 1.5) (drill 0.75) (layers *.Cu *.Mask)
+    (pad "3" smd roundrect (at 0.9375 0 270) (size 1.475 0.6) (layers "F.Cu" "F.Paste" "F.Mask") (roundrect_rratio 0.25)
       (net 23 "/Channel Power Supply 2/Charge Pump/Charge") (pinfunction "C") (pintype "passive"))
-    (model "${KICAD6_3DMODEL_DIR}/Package_TO_SOT_THT.3dshapes/TO-92_Inline.wrl"
-      (offset (xyz 0 0 0))
-      (scale (xyz 1 1 1))
+    (model "${KICAD6_3DMODEL_DIR}/Package_TO_SOT_SMD.3dshapes/SOT-23.wrl"
+      (offset (xyz 0 0 0))
+      (scale (xyz 1 1 1))

Commit message: Update pcb footprints
Parts:
- removed D1_S1, D1_S2, D_5V1: 1N4001, Diode_SMD:D_SMA
- removed J_5V1: Conn_01x01_Male, Connector_PinHeader_2.54mm:PinHeader_1x01_P2.54mm_Vertical
- removed J_FrontPanel1: Conn_02x10_Counter_Clockwise, Connector_IDC:IDC-Header_2x10_P2.54mm_Vertical
- removed L_5V2: 22u, Inductor_THT:L_Radial_D6.0mm_P4.00mm
- removed Linear2_1: LT3080xDD, Package_DFN_QFN:DFN-8-1EP_3x3mm_P0.5mm_EP1.66x2.38mm
- removed Q_CP1, Q_CP2: 2N2219, Package_TO_SOT_SMD:SOT-23
- removed R1_G1, R1_G2, R2_G1, R2_G2, R3_G1, R3_G2: 1k, Resistor_SMD:R_0603_1608Metric
- removed R1_OA1, R1_OA2, R1_S1, R1_S2, R3_SVR1, R3_SVR2, R5_OA1, R5_OA2: 4k, Resistor_SMD:R_0603_1608Metric
- removed R2_CS1, R2_CS2, R9_OA1, R9_OA2: 3k, Resistor_SMD:R_0603_1608Metric
- removed R2_LED1: 100, Resistor_SMD:R_0603_1608Metric
- removed R4_SVR1, R4_SVR2, R8_SVR1, R8_SVR2: 1.2k, Resistor_SMD:R_0603_1608Metric
- removed RotaryEncoder+Switch2: IgnorePinsOnSymbol, Rotary_Encoder:RotaryEncoder_Alps_EC11E-Switch_Vertical_H20mm
- added D_LVR1: 1N4001, Diode_SMD:D_SMA, F.Cu at (185.4, -45.7)
- added D_LVR2: 1N4001, Diode_SMD:D_SMA, F.Cu at (263.6, -89.7)
- added FrontPanel1: Conn_02x10_Counter_Clockwise, Connector_IDC:IDC-Header_2x10_P2.54mm_Vertical, F.Cu at (186.6, -85.8)
- added Linear1_2: LT3080xDD, Package_DFN_QFN:DFN-8-1EP_3x3mm_P0.5mm_EP1.66x2.38mm, F.Cu at (262.1, -85.0)
- added R11_LVR1: 2k, Resistor_SMD:R_0603_1608Metric, F.Cu at (183.4, -39.7)
- added R11_LVR2: 2k, Resistor_SMD:R_0603_1608Metric, F.Cu at (266.6, -86.1)
- added R12_LVR1: 2k, Resistor_SMD:R_0603_1608Metric, F.Cu at (183.4, -42.2)
- added R12_LVR2: 2k, Resistor_SMD:R_0603_1608Metric, F.Cu at (269.6, -90.7)
- added R12_OA1: 2k, Resistor_SMD:R_0603_1608Metric, F.Cu at (233.6, -85.7)
- added R12_OA2: 2k, Resistor_SMD:R_0603_1608Metric, F.Cu at (198.8, -41.7)
- added R13_OA1: 2k, Resistor_SMD:R_0603_1608Metric, F.Cu at (233.6, -83.1)
- added R13_OA2: 2k, Resistor_SMD:R_0603_1608Metric, F.Cu at (198.8, -39.2)
- added R1_LED2: 100, Resistor_SMD:R_0603_1608Metric, F.Cu at (183.4, -55.6)
- added R21_CS1: 2k, Resistor_SMD:R_0603_1608Metric, F.Cu at (247.6, -88.2)
- added R21_CS2: 2k, Resistor_SMD:R_0603_1608Metric, F.Cu at (233.6, -51.0)
- added R22_CS1: 1k, Resistor_SMD:R_0603_1608Metric, F.Cu at (247.6, -90.7)
- added R22_CS2: 1k, Resistor_SMD:R_0603_1608Metric, F.Cu at (233.6, -53.6)
- added R2_LVR1: 0, Resistor_SMD:R_0603_1608Metric, F.Cu at (191.4, -46.7)
- added R2_LVR2: 0, Resistor_SMD:R_0603_1608Metric, F.Cu at (261.5, -81.5)
- added R31_SVR1: 2k, Resistor_SMD:R_0603_1608Metric, F.Cu at (219.6, -90.7)
- added R31_SVR2: 2k, Resistor_SMD:R_0603_1608Metric, F.Cu at (219.6, -53.6)
- added R32_SVR1: 2k, Resistor_SMD:R_0603_1608Metric, F.Cu at (219.6, -85.7)
- added R32_SVR2: 2k, Resistor_SMD:R_0603_1608Metric, F.Cu at (219.6, -48.5)
- added R3_LVR1: 1k, Resistor_SMD:R_0603_1608Metric, F.Cu at (191.4, -44.2)
- added R3_LVR2: 1k, Resistor_SMD:R_0603_1608Metric, F.Cu at (265.6, -81.5)
- added R41_SVR1: 1.2k, Resistor_SMD:R_0603_1608Metric, F.Cu at (219.6, -88.2)
- added R41_SVR2: 1.2k, Resistor_SMD:R_0603_1608Metric, F.Cu at (219.6, -51.0)
- added R42_SVR1: 1.2k, Resistor_SMD:R_0603_1608Metric, F.Cu at (223.6, -90.7)
- added R42_SVR2: 1.2k, Resistor_SMD:R_0603_1608Metric, F.Cu at (223.6, -53.6)
- added R4_LVR1: 1k, Resistor_SMD:R_0603_1608Metric, F.Cu at (187.4, -42.2)
- added R4_LVR2: 1k, Resistor_SMD:R_0603_1608Metric, F.Cu at (261.5, -79.0)
- added R51_OA1: 2k, Resistor_SMD:R_0603_1608Metric, F.Cu at (237.6, -88.2)
- added R51_OA2: 2k, Resistor_SMD:R_0603_1608Metric, F.Cu at (202.8, -44.2)
- added R52_OA1: 2k, Resistor_SMD:R_0603_1608Metric, F.Cu at (237.6, -90.7)
- added R52_OA2: 2k, Resistor_SMD:R_0603_1608Metric, F.Cu at (202.8, -46.7)
- added R91_OA1: 2k, Resistor_SMD:R_0603_1608Metric, F.Cu at (233.6, -90.7)
- added R91_OA2: 2k, Resistor_SMD:R_0603_1608Metric, F.Cu at (198.8, -46.7)
- added R92_OA1: 1k, Resistor_SMD:R_0603_1608Metric, F.Cu at (233.6, -88.2)
- added R92_OA2: 1k, Resistor_SMD:R_0603_1608Metric, F.Cu at (198.8, -44.2)
- C10_Power1, C1_3.3V1, C1_3.3V2, C1_Power1, C1_Power2, C2_Power1, C2_Power2, C3_Power1, C3_Power2, C3_SVR1, C3_SVR2, C4_LVR1, C4_LVR2, C4_Power1, C4_Power2, C4_SVR1, C4_SVR2, C5_Power1, C5_Power2, C6_Power1, C6_Power2, C7_Power1, C7_Power2, C8_Power1, C8_Power2, C9_Power1: footprint Capacitor_SMD:C_0805_2012Metric -> Capacitor_SMD:C_0603_1608Metric
- C1_5V1, C3_5V1: value 100u -> 68u; footprint Capacitor_THT:CP_Radial_D10.0mm_P5.00mm -> Capacitor_THT:CP_Radial_D8.0mm_P3.50mm
- C2_5V1: value 10n -> 100n; footprint Capacitor_SMD:C_0805_2012Metric -> Capacitor_SMD:C_0603_1608Metric
- F_CS1, F_CS2: value 320m -> 290m
- L_5V1: value 22u -> 4.7u; footprint Inductor_THT:L_Radial_D6.0mm_P4.00mm -> Inductor_SMD:L_Sumida_CDMC6D28_7.25x6.5mm
- L_SVR1, L_SVR2: footprint Inductor_THT:L_Radial_D6.0mm_P4.00mm -> Inductor_SMD:L_Sumida_CR75
- U_5V1: value LM2672M-5.0 -> AP63205WU; footprint Package_SO:SOIC-8_3.9x4.9mm_P1.27mm -> Package_TO_SOT_SMD:TSOT-23-6
Connections:
- net /Front Panel/GND renamed Net-(FrontPanel1-Pad5)
- net Net-(MCU_1-Pad7) renamed /Primary Controller/Reset
- C3_5V1 pad 1: /Channel 1 Power Rails/LCD Power -> /Channel 1 Power Rails/5 Volts
- Front_Panel1 pad 1: Net-(Front_Panel1-Pad1) -> +3.3V
- Front_Panel1 pad 12: GND1 -> Net-(Front_Panel1-Pad12)
- Front_Panel1 pad 16: GND1 -> Net-(Front_Panel1-Pad16)
- Front_Panel1 pad 17: Net-(Front_Panel1-Pad17) -> (no net)
- Front_Panel1 pad 18: Net-(Front_Panel1-Pad18) -> (no net)
- Front_Panel1 pad 19: Net-(Front_Panel1-Pad19) -> (no net)
- Front_Panel1 pad 20: +3.3V -> (no net)
- Front_Panel1 pad 5: Net-(Front_Panel1-Pad5) -> GND1
- J_I2C1 pad 1: /Primary Controller/I2C SDA -> GND1
- J_I2C1 pad 2: /Primary Controller/I2C SCL -> /Channel 1 Power Rails/5 Volts
- J_I2C1 pad 3: GND1 -> /Primary Controller/I2C SDA
- J_STLink1 pad 1: /Primary Controller/SWDIO -> +3.3V
- J_STLink1 pad 2: /Primary Controller/SWCLK -> GND1
- J_STLink1 pad 3: GND1 -> /Primary Controller/SWDIO
- J_STLink2 pad 1: Net-(J_STLink2-Pad1) -> +3.3VA
- J_STLink2 pad 2: Net-(J_STLink2-Pad2) -> GND2
- J_STLink2 pad 3: GND2 -> Net-(J_STLink2-Pad3)
- L_5V1 pad 1: Net-(C2_5V1-Pad2) -> Net-(C2_5V1-Pad1)
- L_5V1 pad 2: Net-(L_5V1-Pad2) -> /Channel 1 Power Rails/5 Volts
- Linear1_1 pad 1: unconnected-(Linear1_1-Pad1) -> /Channel Power Supply 1/Charge Pump/Charge
- Linear1_1 pad 2: unconnected-(Linear1_1-Pad2) -> /Channel Power Supply 1/Charge Pump/Charge
- Linear1_1 pad 3: unconnected-(Linear1_1-Pad3) -> /Channel Power Supply 1/Charge Pump/Charge
- Linear1_1 pad 4: unconnected-(Linear1_1-Pad4) -> Net-(C4_LVR1-Pad1)
- Linear1_1 pad 5: unconnected-(Linear1_1-Pad5) -> VCC
- Linear1_1 pad 7: unconnected-(Linear1_1-Pad7) -> /Channel Power Supply 1/Linear Voltage Regulator /Linear Input
- Linear1_1 pad 8: unconnected-(Linear1_1-Pad8) -> /Channel Power Supply 1/Linear Voltage Regulator /Linear Input
- Linear1_1 pad 9: unconnected-(Linear1_1-Pad9) -> /Channel Power Supply 1/Charge Pump/Charge
- MCU_1 pad 26: Net-(Front_Panel1-Pad19) -> Net-(Front_Panel1-Pad2)
- MCU_1 pad 27: Net-(Front_Panel1-Pad18) -> Net-(Front_Panel1-Pad3)
- MCU_1 pad 28: Net-(Front_Panel1-Pad17) -> Net-(Front_Panel1-Pad4)
- MCU_1 pad 29: Net-(Front_Panel1-Pad1) -> Net-(Front_Panel1-Pad16)
- MCU_1 pad 30: Net-(Front_Panel1-Pad2) -> Net-(Front_Panel1-Pad15)
- MCU_1 pad 33: Net-(Front_Panel1-Pad3) -> Net-(Front_Panel1-Pad14)
- MCU_1 pad 34: Net-(Front_Panel1-Pad4) -> Net-(Front_Panel1-Pad13)
- MCU_1 pad 35: Net-(Front_Panel1-Pad5) -> Net-(Front_Panel1-Pad12)
- MCU_1 pad 37: Net-(Front_Panel1-Pad6) -> Net-(Front_Panel1-Pad11)
- MCU_1 pad 38: Net-(Front_Panel1-Pad7) -> Net-(Front_Panel1-Pad10)
- MCU_1 pad 39: Net-(Front_Panel1-Pad8) -> Net-(Front_Panel1-Pad9)
- MCU_1 pad 40: Net-(Front_Panel1-Pad9) -> Net-(Front_Panel1-Pad8)
- MCU_1 pad 55: Net-(Front_Panel1-Pad15) -> Net-(Front_Panel1-Pad6)
- MCU_1 pad 56: Net-(Front_Panel1-Pad14) -> Net-(Front_Panel1-Pad7)
- MCU_1 pad 57: Net-(Front_Panel1-Pad13) -> unconnected-(MCU_1-Pad57)
- MCU_1 pad 61: Net-(Front_Panel1-Pad11) -> unconnected-(MCU_1-Pad61)
- MCU_1 pad 62: Net-(Front_Panel1-Pad10) -> unconnected-(MCU_1-Pad62)
- MCU_2 pad 34: Net-(J_STLink2-Pad1) -> Net-(J_STLink2-Pad3)
- MCU_2 pad 37: Net-(J_STLink2-Pad2) -> Net-(J_STLink2-Pad4)
- Q3_LVR1 pad 3: /Channel Power Supply 1/Charge Pump/Charge -> Net-(D_LVR1-Pad2)
- Q3_LVR2 pad 3: /Channel Power Supply 2/Charge Pump/Charge -> Net-(D_LVR2-Pad2)
- R1_Boot1 pad 1: Net-(J_Boot1-Pad3) -> Net-(J_Boot1-Pad1)
- R1_Boot1 pad 2: GND1 -> +3.3V
- R1_Boot2 pad 1: Net-(J_Boot2-Pad3) -> +3.3VA
- R1_Boot2 pad 2: GND2 -> Net-(J_Boot2-Pad1)
- R2_Boot1 pad 1: Net-(J_Boot1-Pad1) -> Net-(J_Boot1-Pad3)
- R2_Boot1 pad 2: +3.3V -> GND1
- R2_Boot2 pad 1: +3.3VA -> Net-(J_Boot2-Pad3)
- R2_Boot2 pad 2: Net-(J_Boot2-Pad1) -> GND2
- R_CP1 pad 2: Net-(Q_CP1-Pad1) -> unconnected-(R_CP1-Pad2)
- R_CP2 pad 2: Net-(Q_CP2-Pad1) -> unconnected-(R_CP2-Pad2)
- U_5V1 pad 1: Net-(C2_5V1-Pad1) -> /Channel 1 Power Rails/5 Volts
- U_5V1 pad 2: unconnected-(U_5V1-Pad2) -> VCC
- U_5V1 pad 3: unconnected-(U_5V1-Pad3) -> VCC
- U_5V1 pad 4: /Channel 1 Power Rails/LCD Power -> GND1
- U_5V1 pad 5: /Channel 1 Power Rails/3.3 Volt -> Net-(C2_5V1-Pad1)
- U_5V1 pad 6: GND1 -> Net-(C2_5V1-Pad2)
