File: LabPowerSupply/LabPowerSupply.kicad_pcb (KiCad board)
At the start: 4 copper layers, 229 parts, among them Q1_CP1 FMMT495TA, Q1_CP2 FMMT495TA, Q1_LVR1 PJA3404_R1_00001, Q1_LVR2 PJA3404_R1_00001, Q2_LVR1 PJA3404_R1_00001, Q2_LVR2 PJA3404_R1_00001, Q3_LVR1 PJA3404_R1_00001, Q3_LVR2 PJA3404_R1_00001, SW11 Decimal, SW12 0, SW13 Backspace, SW14 Current 2, SW15 Cancel, SW21 1, SW22 2, SW23 3, SW24 Voltage 2, SW25 Confirm, SW31 4, SW32 5, SW33 6, SW34 Current 1, SW35 Channel 2, SW41 7, SW42 8, SW43 9, SW44 Voltage 1, SW45 Channel 1, Y1 8M, Y2 8M

Commit message: Added the Front Panel Project
Parts:
- removed Front_Panel2: Conn_02x08_Counter_Clockwise, Connector_IDC:IDC-Header_2x08_P2.54mm_Vertical
- removed Power1, Power2: LED, LED_THT:LED_D3.0mm
- removed R1_LED1, R1_LED2: 100, Resistor_SMD:R_0603_1608Metric
- removed RotaryEncoder+Switch1: IgnorePinsOnSymbol, Rotary_Encoder:RotaryEncoder_Alps_EC11E-Switch_Vertical_H20mm
- removed SW11: Decimal, Button_Switch_SMD:SW_MEC_5GSH9
- removed SW12: 0, Button_Switch_SMD:SW_MEC_5GSH9
- removed SW13: Backspace, Button_Switch_SMD:SW_MEC_5GSH9
- removed SW14: Current 2, Button_Switch_SMD:SW_MEC_5GSH9
- removed SW15: Cancel, Button_Switch_SMD:SW_MEC_5GSH9
- removed SW21: 1, Button_Switch_SMD:SW_MEC_5GSH9
- removed SW22: 2, Button_Switch_SMD:SW_MEC_5GSH9
- removed SW23: 3, Button_Switch_SMD:SW_MEC_5GSH9
- removed SW24: Voltage 2, Button_Switch_SMD:SW_MEC_5GSH9
- removed SW25: Confirm, Button_Switch_SMD:SW_MEC_5GSH9
- removed SW31: 4, Button_Switch_SMD:SW_MEC_5GSH9
- removed SW32: 5, Button_Switch_SMD:SW_MEC_5GSH9
- removed SW33: 6, Button_Switch_SMD:SW_MEC_5GSH9
- removed SW34: Current 1, Button_Switch_SMD:SW_MEC_5GSH9
- removed SW35: Channel 2, Button_Switch_SMD:SW_MEC_5GSH9
- removed SW41: 7, Button_Switch_SMD:SW_MEC_5GSH9
- removed SW42: 8, Button_Switch_SMD:SW_MEC_5GSH9
- removed SW43: 9, Button_Switch_SMD:SW_MEC_5GSH9
- removed SW44: Voltage 1, Button_Switch_SMD:SW_MEC_5GSH9
- removed SW45: Channel 1, Button_Switch_SMD:SW_MEC_5GSH9
- J_USB1, R_CC1, R_CC2: moved to B.Cu
- SW_Reset1, SW_Reset2: moved to F.Cu
- moved C_3.3V2 57.7 mm to (51.5, 185.6), turned to 0 degrees
- moved Front_Panel1 55.8 mm to (319.5, 139.4)
- moved Input4 53.6 mm to (22.4, 141.2)
- moved D4_BR2 52.6 mm to (29.5, 140.2), turned to -90 degrees
- moved D3_BR2 52.5 mm to (15.7, 140.2), turned to 90 degrees
- moved Input2 50.3 mm to (26.0, 69.6)
- moved U_3.3V2 50.1 mm to (40.1, 180.6)
- moved D4_BR1 49.4 mm to (33.1, 68.6), turned to -90 degrees
- moved D3_BR1 49.3 mm to (19.4, 68.6), turned to 90 degrees
- moved Input1 45.3 mm to (26.0, 25.4)
- moved D2_BR1 44.3 mm to (32.6, 26.4), turned to 90 degrees
- moved D1_BR1 44.2 mm to (19.4, 26.4), turned to -90 degrees
- moved L_5V2 43.1 mm to (46.0, 165.8)
- moved Input3 42.5 mm to (22.4, 97.0)
- moved D2_BR2 41.6 mm to (29.0, 98.0), turned to 90 degrees
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