File: LabPowerSupply/LinearVoltageRegulator.kicad_sch (KiCad schematic)
At the start: 14 parts, among them Q1_LVR1 PJA3404_R1_00001, Q2_LVR1 PJA3404_R1_00001, Q3_LVR1 PJA3404_R1_00001

Commit message: another commit
Parts:
- C3_LVR1, C4_LVR1: footprint Capacitor_THT:C_Disc_D5.0mm_W2.5mm_P2.50mm -> Capacitor_THT:C_Disc_D7.5mm_W2.5mm_P5.00mm
Changed lines of the file:
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@@
       (effects (font (size 1.27 1.27)) (justify left))
     )
-    (property "Footprint" "Capacitor_THT:C_Disc_D5.0mm_W2.5mm_P2.50mm" (id 2) (at 155.9052 111.76 0)
+    (property "Footprint" "Capacitor_THT:C_Disc_D7.5mm_W2.5mm_P5.00mm" (id 2) (at 155.9052 111.76 0)
       (effects (font (size 1.27 1.27)) hide)
     )
@@
     (property "Reference" "C4_LVR1" (id 0) (at 175.26 106.68 0))
     (property "Value" "100n" (id 1) (at 175.26 109.22 0))
-    (property "Footprint" "Capacitor_THT:C_Disc_D5.0mm_W2.5mm_P2.50mm" (id 2) (at 169.8752 111.76 0)
+    (property "Footprint" "Capacitor_THT:C_Disc_D7.5mm_W2.5mm_P5.00mm" (id 2) (at 169.8752 111.76 0)
       (effects (font (size 1.27 1.27)) hide)
     )

Commit message: fixed linear cap footprints
Parts:
- C3_LVR1, C4_LVR1: footprint Capacitor_THT:C_Disc_D7.5mm_W2.5mm_P5.00mm -> (none)
Changed lines of the file:
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@@
       (effects (font (size 1.27 1.27)) (justify left))
     )
-    (property "Footprint" "Capacitor_THT:C_Disc_D7.5mm_W2.5mm_P5.00mm" (id 2) (at 155.9052 111.76 0)
+    (property "Footprint" "" (id 2) (at 155.9052 111.76 0)
       (effects (font (size 1.27 1.27)) hide)
     )
@@
     (property "Reference" "C4_LVR1" (id 0) (at 175.26 106.68 0))
     (property "Value" "100n" (id 1) (at 175.26 109.22 0))
-    (property "Footprint" "Capacitor_THT:C_Disc_D7.5mm_W2.5mm_P5.00mm" (id 2) (at 169.8752 111.76 0)
+    (property "Footprint" "" (id 2) (at 169.8752 111.76 0)
       (effects (font (size 1.27 1.27)) hide)
     )

Commit message: Changed most parts to smd
Parts:
- added Linear1_1: LT3080xDD, Package_DFN_QFN:DFN-8-1EP_3x3mm_P0.5mm_EP1.66x2.38mm, symbol Regulator_Linear:LT3080xDD
- C1_LVR1, C2_LVR1: footprint Capacitor_THT:C_Disc_D5.0mm_W2.5mm_P2.50mm -> Capacitor_SMD:C_0805_2012Metric
- C3_LVR1, C4_LVR1: footprint (none) -> Capacitor_SMD:C_0805_2012Metric
- D1_S1: value SB130 -> 1N4001; footprint Diode_THT:D_DO-41_SOD81_P10.16mm_Horizontal -> Diode_SMD:D_SMA; symbol Diode:SB130 -> Diode:1N4001
- Inverter1: footprint Package_DIP:DIP-14_W7.62mm -> Package_SO:SSOP-14_5.3x6.2mm_P0.65mm
Changed lines of the file:
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@@
       (effects (font (size 1.27 1.27)) (justify left))
     )
-    (property "Footprint" "Package_DIP:DIP-14_W7.62mm" (id 2) (at 82.55 102.87 0)
+    (property "Footprint" "Package_SO:SSOP-14_5.3x6.2mm_P0.65mm" (id 2) (at 82.55 102.87 0)
       (effects (font (size 1.27 1.27)) hide)
     )
@@
     (property "Reference" "Inverter1" (id 0) (at 162.56 60.96 0))
     (property "Value" "74AHC04" (id 1) (at 162.56 63.5 0))
-    (property "Footprint" "Package_DIP:DIP-14_W7.62mm" (id 2) (at 162.56 68.58 0)
+    (property "Footprint" "Package_SO:SSOP-14_5.3x6.2mm_P0.65mm" (id 2) (at 162.56 68.58 0)
       (effects (font (size 1.27 1.27)) hide)
     )
@@
     (property "Reference" "C1_LVR1" (id 0) (at 115.57 87.63 90))
     (property "Value" "4.7u" (id 1) (at 115.57 90.17 90))
-    (property "Footprint" "Capacitor_THT:C_Disc_D5.0mm_W2.5mm_P2.50mm" (id 2) (at 119.38 94.2848 0)
+    (property "Footprint" "Capacitor_SMD:C_0805_2012Metric" (id 2) (at 119.38 94.2848 0)
       (effects (font (size 1.27 1.27)) hide)
     )
@@
       (effects (font (size 1.27 1.27)) (justify left))
     )
-    (property "Footprint" "" (id 2) (at 155.9052 111.76 0)
+    (property "Footprint" "Capacitor_SMD:C_0805_2012Metric" (id 2) (at 155.9052 111.76 0)
       (effects (font (size 1.27 1.27)) hide)
     )
@@
     (pin "2")
   )
-  (symbol (lib_id "Diode:SB130") (at 171.45 95.25 0) (unit 1)
-    (in_bom yes) (on_board yes) (fields_autoplaced)
+  (symbol (lib_id "Diode:1N4001") (at 171.45 95.25 0) (unit 1)
+    (in_bom yes) (on_board yes)
     (property "Reference" "D1_S1" (id 0) (at 171.1325 88.9 0))
-    (property "Value" "SB130" (id 1) (at 171.1325 91.44 0))
-    (property "Footprint" "Diode_THT:D_DO-41_SOD81_P10.16mm_Horizontal" (id 2) (at 171.45 99.695 0)
-      (effects (font (size 1.27 1.27)) hide)
-    )
-    (property "Datasheet" "http://www.diodes.com/_files/datasheets/ds23022.pdf" (id 3) (at 171.45 95.25 0)
+    (property "Value" "1N4001" (id 1) (at 171.45 91.44 0))
+    (property "Footprint" "Diode_SMD:D_SMA" (id 2) (at 171.45 99.695 0)
+      (effects (font (size 1.27 1.27)) hide)
+    )
+    (property "Datasheet" "http://www.vishay.com/docs/88503/1n4001.pdf" (id 3) (at 171.45 95.25 0)
       (effects (font (size 1.27 1.27)) hide)
     )
@@
     (property "Reference" "C4_LVR1" (id 0) (at 175.26 106.68 0))
     (property "Value" "100n" (id 1) (at 175.26 109.22 0))
-    (property "Footprint" "" (id 2) (at 169.8752 111.76 0)
+    (property "Footprint" "Capacitor_SMD:C_0805_2012Metric" (id 2) (at 169.8752 111.76 0)
       (effects (font (size 1.27 1.27)) hide)
     )
@@
     (pin "1")
     (pin "2")
+  )
+  (symbol (lib_id "Regulator_Linear:LT3080xDD") (at 138.43 132.08 0) (unit 1)
+    (in_bom yes) (on_board yes) (fields_autoplaced)
+    (property "Reference" "Linear1_1" (id 0) (at 138.43 119.38 0))
+    (property "Value" "LT3080xDD" (id 1) (at 138.43 121.92 0))
+    (property "Footprint" "Package_DFN_QFN:DFN-8-1EP_3x3mm_P0.5mm_EP1.66x2.38mm" (id 2) (at 138.43 142.24 0)
+      (effects (font (size 1.27 1.27)) hide)
+    )
+    (property "Datasheet" "https://www.analog.com/media/en/technical-documentation/data-sheets/3080fc.pdf" (id 3) (at 94.742 112.522 0)
+      (effects (font (size 1.27 1.27)) hide)
+    )
+    (pin "1")
+    (pin "2")
+    (pin "3")
+    (pin "4")
+    (pin "5")
+    (pin "6")
+    (pin "7")
+    (pin "8")
+    (pin "9")
   )
   (symbol (lib_id "Device:C") (at 118.11 107.95 0) (unit 1)
@@
       (effects (font (size 1.27 1.27)) (justify left))
     )
-    (property "Footprint" "Capacitor_THT:C_Disc_D5.0mm_W2.5mm_P2.50mm" (id 2) (at 119.0752 111.76 0)
-      (effects (font (size 1.27 1.27)) hide)
-    )
+    (property "Footprint" "Capacitor_SMD:C_0805_2012Metric" (id 2) (at 119.0752 111.76 0)
+      (effects (font (size 1.27 1.27)) hide)
+    )

Commit message: almost done
Parts:
- removed C1_LVR1: 4.7u, Capacitor_SMD:C_0805_2012Metric, symbol Device:C
- removed C2_LVR1, C3_LVR1: 10u, Capacitor_SMD:C_0805_2012Metric, symbol Device:C
- removed C4_LVR1: 100n, Capacitor_SMD:C_0805_2012Metric, symbol Device:C
- removed D1_S1: 1N4001, Diode_SMD:D_SMA, symbol Diode:1N4001
- removed Inverter1: 74AHC04, Package_SO:SSOP-14_5.3x6.2mm_P0.65mm, symbol 74xx:74AHC04
- removed Linear1: LT3083ET#PBF, SamacSys_Parts:TO170P457X1022X2306-5P, symbol SamacSys_Parts:LT3083ET#PBF
- removed Linear1_1: LT3080xDD, Package_DFN_QFN:DFN-8-1EP_3x3mm_P0.5mm_EP1.66x2.38mm, symbol Regulator_Linear:LT3080xDD
- removed Q1_LVR1, Q2_LVR1, Q3_LVR1: PJA3404_R1_00001, SamacSys_Parts:SOT95P240X110-3N, symbol SamacSys_Parts:PJA3404_R1_00001
- removed R1_G1, R2_G1, R3_G1: 1k, Resistor_SMD:R_0603_1608Metric, symbol Device:R_US
- removed R1_S1: 4k, Resistor_SMD:R_0603_1608Metric, symbol Device:R_US
- added C1_LVR2: 4.7u, Capacitor_SMD:C_0805_2012Metric, symbol Device:C
- added C2_LVR2, C3_LVR2: 10u, Capacitor_SMD:C_0805_2012Metric, symbol Device:C
- added C4_LVR2: 100n, Capacitor_SMD:C_0603_1608Metric, symbol Device:C
- added D_LVR2: 1N4001, Diode_SMD:D_SMA, symbol Diode:1N4001
- added Inverter2: 74AHC04, Package_SO:SSOP-14_5.3x6.2mm_P0.65mm, symbol 74xx:74AHC04
- added Linear1_2: LT3080xDD, Package_DFN_QFN:DFN-8-1EP_3x3mm_P0.5mm_EP1.66x2.38mm, symbol Regulator_Linear:LT3080xDD
- added Linear2: LT3083ET#PBF, SamacSys_Parts:TO170P457X1022X2306-5P, symbol SamacSys_Parts:LT3083ET#PBF
- added Q1_LVR2, Q2_LVR2, Q3_LVR2: PJA3404_R1_00001, SamacSys_Parts:SOT95P240X110-3N, symbol SamacSys_Parts:PJA3404_R1_00001
- added R11_LVR2, R12_LVR2: 2k, Resistor_SMD:R_0603_1608Metric, symbol Device:R_US
- added R2_LVR2: 0, Resistor_SMD:R_0603_1608Metric, symbol Device:R_US
- added R3_LVR2, R4_LVR2: 1k, Resistor_SMD:R_0603_1608Metric, symbol Device:R_US
Connections:
- net 3.3 Volts: now also Inverter2.14 (VCC)
- net Charge: now also C3_LVR2.1, Linear1_2.1 (OUT), Linear1_2.2 (OUT), Linear1_2.3 (OUT), Linear1_2.9 (OUT), Linear2.3 (OUT)
- net GND: now also C1_LVR2.1, C2_LVR2.2, C3_LVR2.2, C4_LVR2.2, Inverter2.7 (GND), Q2_LVR2.2 (S), Q3_LVR2.2 (S)
- net Linear Input: now also C2_LVR2.1, Linear1_2.7 (IN), Linear1_2.8 (IN), Linear2.5 (IN)
- net On/Off: now also Inverter2.1, R3_LVR2.2, R4_LVR2.2
- net Set Voltage: now also Q1_LVR2.3 (D)
- net VCC: now also C1_LVR2.2, Linear1_2.5 (VCONTROL), Linear2.4 (VCONTROL)
- new net: C4_LVR2.1, D_LVR2.1 (K), Linear1_2.4 (SET), Linear2.2 (SET), R12_LVR2.1
- new net: R11_LVR2.1, R12_LVR2.2
- new net: Q1_LVR2.1 (G), R2_LVR2.1
- new net: Inverter2.2, R2_LVR2.2
- new net: Q1_LVR2.2 (S), Q2_LVR2.3 (D), R11_LVR2.2
- new net: Q2_LVR2.1 (G), R3_LVR2.1
- new net: Q3_LVR2.1 (G), R4_LVR2.1
- new net: D_LVR2.2 (A), Q3_LVR2.3 (D)

Commit message: Update pcb footprints
Parts:
- renumbered C1_LVR2 to C1_LVR1, C2_LVR2 to C2_LVR1, C3_LVR2 to C3_LVR1, C4_LVR2 to C4_LVR1, D_LVR2 to D_LVR1, Inverter2 to Inverter1, Linear2 to Linear1, Linear1_2 to Linear1_1, Q1_LVR2 to Q1_LVR1, Q2_LVR2 to Q2_LVR1, Q3_LVR2 to Q3_LVR1, R11_LVR2 to R11_LVR1, R12_LVR2 to R12_LVR1, R2_LVR2 to R2_LVR1, R3_LVR2 to R3_LVR1, R4_LVR2 to R4_LVR1
Changed lines of the file:
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@@
   (symbol (lib_id "Device:R_US") (at 173.99 114.3 180) (unit 1)
     (in_bom yes) (on_board yes) (fields_autoplaced)
-    (property "Reference" "R12_LVR2" (id 0) (at 176.53 113.0299 0)
+    (property "Reference" "R12_LVR1" (id 0) (at 176.53 113.0299 0)
       (effects (font (size 1.27 1.27)) (justify right))
     )
@@
   (symbol (lib_id "74xx:74AHC04") (at 97.79 127 0) (unit 7)
     (in_bom yes) (on_board yes) (fields_autoplaced)
-    (property "Reference" "Inverter2" (id 0) (at 104.14 125.7299 0)
+    (property "Reference" "Inverter1" (id 0) (at 104.14 125.7299 0)
       (effects (font (size 1.27 1.27)) (justify left))
     )
@@
   (symbol (lib_id "Device:C") (at 184.15 132.08 0) (unit 1)
     (in_bom yes) (on_board yes)
-    (property "Reference" "C4_LVR2" (id 0) (at 190.5 130.81 0))
+    (property "Reference" "C4_LVR1" (id 0) (at 190.5 130.81 0))
     (property "Value" "100n" (id 1) (at 190.5 133.35 0))
     (property "Footprint" "Capacitor_SMD:C_0603_1608Metric" (id 2) (at 185.1152 135.89 0)
@@
   (symbol (lib_id "Device:R_US") (at 163.83 69.85 90) (unit 1)
     (in_bom yes) (on_board yes) (fields_autoplaced)
-    (property "Reference" "R2_LVR2" (id 0) (at 163.83 63.5 90))
+    (property "Reference" "R2_LVR1" (id 0) (at 163.83 63.5 90))
     (property "Value" "0" (id 1) (at 163.83 66.04 90))
     (property "Footprint" "Resistor_SMD:R_0603_1608Metric" (id 2) (at 164.084 68.834 90)
@@
   (symbol (lib_id "Device:R_US") (at 173.99 102.87 180) (unit 1)
     (in_bom yes) (on_board yes) (fields_autoplaced)
-    (property "Reference" "R11_LVR2" (id 0) (at 176.53 101.5999 0)
+    (property "Reference" "R11_LVR1" (id 0) (at 176.53 101.5999 0)
       (effects (font (size 1.27 1.27)) (justify right))
     )
@@
   (symbol (lib_id "SamacSys_Parts:LT3083ET#PBF") (at 170.18 119.38 0) (mirror y) (unit 1)
     (in_bom yes) (on_board yes) (fields_autoplaced)
-    (property "Reference" "Linear2" (id 0) (at 153.67 111.76 0))
+    (property "Reference" "Linear1" (id 0) (at 153.67 111.76 0))
     (property "Value" "LT3083ET#PBF" (id 1) (at 153.67 114.3 0))
     (property "Footprint" "SamacSys_Parts:TO170P457X1022X2306-5P" (id 2) (at 140.97 116.84 0)
@@
   (symbol (lib_id "Device:C") (at 130.81 119.38 90) (unit 1)
     (in_bom yes) (on_board yes) (fields_autoplaced)
-    (property "Reference" "C1_LVR2" (id 0) (at 130.81 111.76 90))
+    (property "Reference" "C1_LVR1" (id 0) (at 130.81 111.76 90))
     (property "Value" "4.7u" (id 1) (at 130.81 114.3 90))
     (property "Footprint" "Capacitor_SMD:C_0805_2012Metric" (id 2) (at 134.62 118.4148 0)
@@
   (symbol (lib_id "SamacSys_Parts:PJA3404_R1_00001") (at 204.47 87.63 0) (mirror y) (unit 1)
     (in_bom yes) (on_board yes) (fields_autoplaced)
-    (property "Reference" "Q2_LVR2" (id 0) (at 194.31 80.01 0))
+    (property "Reference" "Q2_LVR1" (id 0) (at 194.31 80.01 0))
     (property "Value" "PJA3404_R1_00001" (id 1) (at 194.31 82.55 0))
     (property "Footprint" "SamacSys_Parts:SOT95P240X110-3N" (id 2) (at 187.96 85.09 0)
@@
   (symbol (lib_id "SamacSys_Parts:PJA3404_R1_00001") (at 214.63 121.92 0) (mirror y) (unit 1)
     (in_bom yes) (on_board yes) (fields_autoplaced)
-    (property "Reference" "Q3_LVR2" (id 0) (at 204.47 114.3 0))
+    (property "Reference" "Q3_LVR1" (id 0) (at 204.47 114.3 0))
     (property "Value" "PJA3404_R1_00001" (id 1) (at 204.47 116.84 0))
     (property "Footprint" "SamacSys_Parts:SOT95P240X110-3N" (id 2) (at 198.12 119.38 0)
@@
   (symbol (lib_id "Device:R_US") (at 214.63 95.25 180) (unit 1)
     (in_bom yes) (on_board yes) (fields_autoplaced)
-    (property "Reference" "R4_LVR2" (id 0) (at 217.17 93.9799 0)
+    (property "Reference" "R4_LVR1" (id 0) (at 217.17 93.9799 0)
       (effects (font (size 1.27 1.27)) (justify right))
     )
@@
   (symbol (lib_id "Regulator_Linear:LT3080xDD") (at 153.67 100.33 0) (unit 1)
     (in_bom yes) (on_board yes)
-    (property "Reference" "Linear1_2" (id 0) (at 153.67 87.63 0))
+    (property "Reference" "Linear1_1" (id 0) (at 153.67 87.63 0))
     (property "Value" "LT3080xDD" (id 1) (at 153.67 90.17 0))
     (property "Footprint" "Package_DFN_QFN:DFN-8-1EP_3x3mm_P0.5mm_EP1.66x2.38mm" (id 2) (at 153.67 110.49 0)
@@
   (symbol (lib_id "SamacSys_Parts:PJA3404_R1_00001") (at 157.48 69.85 0) (mirror y) (unit 1)
     (in_bom yes) (on_board yes) (fields_autoplaced)
-    (property "Reference" "Q1_LVR2" (id 0) (at 147.32 62.23 0))
+    (property "Reference" "Q1_LVR1" (id 0) (at 147.32 62.23 0))
     (property "Value" "PJA3404_R1_00001" (id 1) (at 147.32 64.77 0))
     (property "Footprint" "SamacSys_Parts:SOT95P240X110-3N" (id 2) (at 140.97 67.31 0)
@@
   (symbol (lib_id "Diode:1N4001") (at 187.96 121.92 0) (unit 1)
     (in_bom yes) (on_board yes)
-    (property "Reference" "D_LVR2" (id 0) (at 187.6425 115.57 0))
+    (property "Reference" "D_LVR1" (id 0) (at 187.6425 115.57 0))
     (property "Value" "1N4001" (id 1) (at 187.96 118.11 0))
     (property "Footprint" "Diode_SMD:D_SMA" (id 2) (at 187.96 126.365 0)
@@
   (symbol (lib_id "Device:R_US") (at 204.47 77.47 180) (unit 1)
     (in_bom yes) (on_board yes) (fields_autoplaced)
-    (property "Reference" "R3_LVR2" (id 0) (at 207.01 76.1999 0)
+    (property "Reference" "R3_LVR1" (id 0) (at 207.01 76.1999 0)
       (effects (font (size 1.27 1.27)) (justify right))
     )
@@
   (symbol (lib_id "Device:C") (at 133.35 132.08 0) (unit 1)
     (in_bom yes) (on_board yes)
-    (property "Reference" "C2_LVR2" (id 0) (at 137.16 130.8099 0)
+    (property "Reference" "C2_LVR1" (id 0) (at 137.16 130.8099 0)
       (effects (font (size 1.27 1.27)) (justify left))
     )
@@
   (symbol (lib_id "74xx:74AHC04") (at 177.8 69.85 0) (mirror y) (unit 1)
     (in_bom yes) (on_board yes)
-    (property "Reference" "Inverter2" (id 0) (at 177.8 62.23 0))
+    (property "Reference" "Inverter1" (id 0) (at 177.8 62.23 0))
     (property "Value" "74AHC04" (id 1) (at 177.8 64.77 0))
     (property "Footprint" "Package_SO:SSOP-14_5.3x6.2mm_P0.65mm" (id 2) (at 177.8 69.85 0)
@@
   (symbol (lib_id "Device:C") (at 170.18 132.08 0) (unit 1)
     (in_bom yes) (on_board yes) (fields_autoplaced)
-    (property "Reference" "C3_LVR2" (id 0) (at 173.99 130.8099 0)
-      (effects (font (size 1.27 1.27)) (justify left))
-    )
+    (property "Reference" "C3_LVR1" (id 0) (at 173.99 130.8099 0)
+      (effects (font (size 1.27 1.27)) (justify left))
+    )
