File: LabPowerSupply/FrontPanel.kicad_sch (KiCad schematic)
At the start: 26 parts, among them SW11 Decimal, SW12 0, SW13 Backspace, SW14 Current 2, SW15 Cancel, SW21 1, SW22 2, SW23 3, SW24 Voltage 2, SW25 Confirm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

Commit message: removed transformer and bug squached
Parts:
- Front_Panel2: renamed from FrontPanel1; value Conn_02x10_Counter_Clockwise -> Conn_02x08_Counter_Clockwise; footprint Connector_IDC:IDC-Header_2x10_P2.54mm_Vertical -> Connector_IDC:IDC-Header_2x08_P2.54mm_Vertical
Changed lines of the file:
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@@
   (symbol (lib_id "Connector_Generic:Conn_02x08_Counter_Clockwise") (at 116.84 123.19 0) (unit 1)
     (in_bom yes) (on_board yes)
-    (property "Reference" "FrontPanel1" (id 0) (at 118.11 109.22 0))
-    (property "Value" "Conn_02x10_Counter_Clockwise" (id 1) (at 118.11 111.76 0))
-    (property "Footprint" "Connector_IDC:IDC-Header_2x10_P2.54mm_Vertical" (id 2) (at 116.84 123.19 0)
+    (property "Reference" "Front_Panel2" (id 0) (at 118.11 109.22 0))
+    (property "Value" "Conn_02x08_Counter_Clockwise" (id 1) (at 118.11 111.76 0))
+    (property "Footprint" "Connector_IDC:IDC-Header_2x08_P2.54mm_Vertical" (id 2) (at 116.84 123.19 0)
       (effects (font (size 1.27 1.27)) hide)
     )
