File: LabPowerSupply2/CurrentSense.kicad_sch (KiCad schematic)
At the start: 10 parts

Commit message: Updated Version 2
Parts:
- OpAmp1: value LM324A -> LM324
- R2_CS1, R3_CS1, R4_CS1: footprint (none) -> Resistor_SMD:R_0603_1608Metric
Changed lines of the file:
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@@
   (title_block
     (title "Current and Voltage Sensing")
-    (date "2022-09-26")
-    (rev "2")
+    (date "2022-11-16")
+    (rev "3")
     (company "George Mason University")
     (comment 1 "voltage, and a fuse for reverse polarity protection")
@@
       (effects (font (size 1.27 1.27)) (justify left))
     )
-    (property "Value" "LM324A" (id 1) (at 163.83 95.2499 90)
+    (property "Value" "LM324" (id 1) (at 163.83 95.2499 90)
       (effects (font (size 1.27 1.27)) (justify left))
     )
@@
       (effects (font (size 1.27 1.27)) (justify left))
     )
-    (property "Footprint" "" (id 2) (at 158.496 106.934 90)
+    (property "Footprint" "Resistor_SMD:R_0603_1608Metric" (id 2) (at 158.496 106.934 90)
       (effects (font (size 1.27 1.27)) hide)
     )
@@
       (effects (font (size 1.27 1.27)) (justify left))
     )
-    (property "Footprint" "" (id 2) (at 158.496 115.824 90)
+    (property "Footprint" "Resistor_SMD:R_0603_1608Metric" (id 2) (at 158.496 115.824 90)
       (effects (font (size 1.27 1.27)) hide)
     )
@@
       (effects (font (size 1.27 1.27)) (justify left))
     )
-    (property "Footprint" "" (id 2) (at 158.496 128.524 90)
-      (effects (font (size 1.27 1.27)) hide)
-    )
+    (property "Footprint" "Resistor_SMD:R_0603_1608Metric" (id 2) (at 158.496 128.524 90)
+      (effects (font (size 1.27 1.27)) hide)
+    )

Commit message: Beautifing the Schematic
Connections:
- net 3.3 Volt: now also C_CUR1.1; no longer C_CUR1.2
- net ADC 2: now also R3_CS1.1, R4_CS1.2; no longer R3_CS1.2, R4_CS1.1
- net GND: now also C_CUR1.2, R4_CS1.1; no longer C_CUR1.1, R4_CS1.2
- net at OpAmp1.13 (-), OpAmp1.14: now also R2_CS1.2; no longer R2_CS1.1
- new net: R2_CS1.1, R3_CS1.2
Other:
- note added: "Buffering the Output Voltage before the resistor divider will imporve accuracy and efficiency."
- moved on the sheet: C_CUR1, CurrentSense1, D_CS1, F_CS1, OpAmp1D, Output1, R1_CS1, R2_CS1, R3_CS1, R4_CS1
