File: LabPowerSupply2/DifferentialOpAmpCircuit.kicad_sch (KiCad schematic)
At the start: 14 parts

Commit message: Updated Version 2
Parts:
- R13_OA1, R51_OA1: value 2k -> 1k
- R2_OA1: value 1k -> 470
Changed lines of the file:
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@@
   (title_block
     (title "Differential Op-Amp Circuit")
-    (date "2022-09-12")
-    (rev "1")
+    (date "2022-11-16")
+    (rev "2")
     (company "George Mason University")
     (comment 1 "LT3083, this value is currently set to 2.5 volts.")
@@
       (effects (font (size 1.27 1.27)) (justify left))
     )
-    (property "Value" "1k" (id 1) (at 114.3 99.0599 0)
+    (property "Value" "470" (id 1) (at 114.3 99.0599 0)
       (effects (font (size 1.27 1.27)) (justify left))
     )
@@
       (effects (font (size 1.27 1.27)) (justify left))
     )
-    (property "Value" "2k" (id 1) (at 139.7 109.2199 0)
+    (property "Value" "1k" (id 1) (at 139.7 109.2199 0)
       (effects (font (size 1.27 1.27)) (justify left))
     )
@@
     (in_bom yes) (on_board yes)
     (property "Reference" "R13_OA1" (id 0) (at 99.06 77.47 90))
-    (property "Value" "2k" (id 1) (at 100.33 80.01 90))
+    (property "Value" "1k" (id 1) (at 100.33 80.01 90))
     (property "Footprint" "Resistor_SMD:R_0603_1608Metric" (id 2) (at 100.584 82.804 90)
       (effects (font (size 1.27 1.27)) hide)

Commit message: Beautifing the Schematic
Other:
- moved on the sheet: OpAmp1A, OpAmp1B, OpAmp1C, OpAmp1E, R10_OA1, R12_OA1, R13_OA1, R2_OA1, R3_OA1, R4_OA1, R51_OA1, R52_OA1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
