File: LabPowerSupply2/SecondaryController.kicad_sch (KiCad schematic)
At the start: 22 parts, among them Y2 8M

Commit message: Beautifing the Schematic
Parts:
- removed A1_2, D1_2, D2_2: Conn_01x01_Male, symbol Connector:Conn_01x01_Male
- removed ADC342_2: Conn_01x03_Male, Connector_PinHeader_2.54mm:PinHeader_1x03_P2.54mm_Vertical, symbol Connector:Conn_01x03_Male
Connections:
- net GND: no longer C1_Y2.1, C2_Y2.1
- net at J_STLink2.5 (Pin_5), MCU_2.7 (NRST), R_Reset2.2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: now also C1_Y2.1, C2_Y2.1
Other:
- note added: "Bypass Capasitors to be placed besides power pins"
- moved on the sheet: C1_Power2, C1_Y2, C2_Power2, C2_Y2, C3_Power2, C4_Power2, C5_Power2, C6_Power2, C7_Power2, C8_Power2, J_Boot2, J_STLink2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
